File: ctt.sch (KiCad schematic (older format))
At the start: 5 parts, among them CN1 CONN_3, CN2 CONN_3, SW1 SPST, SW1b SPST

Commit message: 2011.04.20-i állapot.
Connections:
- net labels removed: +5V, -5V, GNDPWR
- wire segments 133 -> 122
Other:
- moved on the sheet: CN1, F1, SW1

Commit message: 2011. 05. 01-i állapot.
Connections:
- net labels added: +5V, -5V, 36ú, 37ú, GNDPWR
- net labels removed: 36, 37, 58
- wire segments 122 -> 125
Other:
- moved on the sheet: CN1, F1, SW1

Commit message: 2011. 05. 15. esti állapot.
Parts:
- added SW?: SWITCH_INV, symbol SWITCH_INV
Connections:
- net labels removed: +5V, -5V
- wire segments 125 -> 144
Other:
- moved on the sheet: CN1, F1, SW1

Commit message: 2011.04.16-i állapot.
Parts:
- removed F1: 000 mA, symbol FUSE
- removed SW1, SW1b: SPST, symbol SPST
- added L?: INDUCTOR, symbol INDUCTOR
- added SW? (x3): SWITCH_INV, symbol SWITCH_INV
Connections:
- net 26: now also L?.2
- net CTT/PS1/+Um1: now also SW?.2
- net CTT/PS1/-Um1: now also SW?.2
- net CTT/PS1/POL: now also L?.1
- net CTT/PS2/+Um3: now also SW?.1
- net CTT/PS2/-Um3: now also SW?.3
- net CTT/PS3/+Um2: now also SW?.1
- net CTT/PS3/-Um2: now also SW?.3
- net GND: no longer CN1.2 (PM)
- net 39 renamed CTT/PS4/230V AC
- net 40 renamed CTT/PS4/230V AC
- new net: SW?.1, SW?.3 (x2)
- new net CTT/PS4/PRT GND: CN1.2 (PM)
Other:
- note removed: "Power"
- moved on the sheet: CN1, SW?
