File: ctt.sch (KiCad schematic (older format))
At the start: 7 parts, among them CN1 CONN_3, CN2 CONN_3, J1 INDUCTOR

Commit message: 07.28-i állapot.
Parts:
- removed J1: INDUCTOR, symbol INDUCTOR
- added J1: RELAY, symbol RELAY
Connections:
- net labels removed: 79
- wire segments 233 -> 230

Commit message: 08.07-i állapot.
Connections:
- net labels added: 80
- wire segments 230 -> 220

Commit message: 2012.01.08-i állapot.
Parts:
- removed JC3, JC4: SWITCH_INV, symbol SWITCH_INV
Connections:
- net labels removed: 60, 61, 62, 63, 78, 80
- wire segments 220 -> 209
Other:
- moved on the sheet: JC1, JC2
Changed lines of the file:
@@
-EESchema Schematic File Version 2  date 2011. aug. 11., csütörtök, 07.58.42 CEST
+EESchema Schematic File Version 2  date 2012.01.08. 14:43:31
 LIBS:power
 LIBS:device
@@
 Sheet 1 11
 Title "CTT Transistor tester"
-Date "11 aug 2011"
+Date "8 jan 2012"
 Rev "1.0"
 Comp "Pozsar Zsolt"
@@
 Comment4 ""
 $EndDescr
-Text Label 4650 4750 0    60   ~ 0
-80
-Wire Wire Line
-	4550 4750 4800 4750
+Connection ~ 6550 5800
+Wire Wire Line
+	6100 5800 6550 5800
+Wire Wire Line
+	3250 6600 950  6600
+Wire Wire Line
+	4550 4450 4800 4450
+Wire Wire Line
+	6300 6600 6300 7000
+Wire Wire Line
+	6300 6600 6100 6600
 Wire Wire Line
 	1075 5450 750  5450
@@
 	2025 7400 2150 7400
 Wire Wire Line
-	2150 7400 2150 7500
-Wire Wire Line
-	2150 7500 2750 7500
-Wire Wire Line
-	2750 7500 2750 7100
-Wire Wire Line
-	2750 7100 6600 7100
+	2150 7400 2150 7100
+Wire Wire Line
+	2150 7100 6600 7100
 Wire Wire Line
 	975  5150 975  5050
@@
 Wire Wire Line
 	7300 6350 6600 6350
-Wire Wire Line
-	950  7100 1400 7100
 Connection ~ 1100 5675
 Wire Wire Line
@@
 	6350 3300 6100 3300
 Wire Wire Line
-	1100 5675 1100 6075
-Wire Wire Line
-	1100 6075 1375 6075
-Wire Wire Line
-	6200 7175 6200 6600
-Wire Wire Line
-	6200 7175 2325 7175
+	1100 5675 1100 6050
+Wire Wire Line
+	1100 6050 1375 6050
 Wire Wire Line
 	7300 6600 6400 6600
@@
 	6400 6600 6400 7300
 Wire Wire Line
-	6400 7300 2650 7300
-Wire Wire Line
-	2650 7300 2650 5750
-Wire Wire Line
-	2650 5750 2300 5750
-Wire Wire Line
-	2325 6825 2750 6825
-Wire Wire Line
-	6200 6600 6100 6600
-Wire Wire Line
-	3250 6600 2750 6600
-Wire Wire Line
-	2750 6600 2750 6825
+	6400 7300 2700 7300
+Wire Wire Line
+	2700 7300 2700 5775
+Wire Wire Line
+	2700 5775 2375 5775
 Wire Wire Line
 	4650 3850 4650 3400
@@
 Wire Wire Line
 	6550 4050 6550 6250
-Wire Wire Line
-	6550 6250 7300 6250
 Wire Wire Line
 	4800 6600 4550 6600
@@
 Connection ~ 4675 6600
 Wire Wire Line
-	3250 6500 2700 6500
-Wire Wire Line
-	2700 6500 2700 6675
-Wire Wire Line
-	6300 6500 6300 7025
-Wire Wire Line
-	6300 6500 6100 6500
-Wire Wire Line
-	2700 6675 2325 6675
-Wire Wire Line
 	7300 6500 6500 6500
 Wire Wire Line
@@
 	2600 7400 2600 6150
 Wire Wire Line
-	2600 6150 2300 6150
-Wire Wire Line
-	1375 5825 1150 5825
-Wire Wire Line
-	1150 5825 1150 6225
+	2600 6150 2375 6150
+Wire Wire Line
+	1375 5875 1150 5875
+Wire Wire Line
+	1150 5875 1150 6250
 Wire Wire Line
 	6100 3200 6350 3200
@@
 Wire Bus Line
 	6150 4200 850  4200
-Wire Bus Line
-	850  4200 850  7000
 Wire Wire Line
 	6350 3100 6100 3100
 Wire Wire Line
-	950  6225 1375 6225
-Wire Wire Line
-	1400 6750 950  6750
+	950  6250 1375 6250
 Connection ~ 3000 3950
 Wire Wire Line
-	6300 7025 2325 7025
-Wire Wire Line
 	6600 6350 6600 7100
 Wire Wire Line
@@
 Wire Wire Line
 	2850 1750 2550 1750
-Connection ~ 1150 6225
+Connection ~ 1150 6250
 Wire Wire Line
 	2950 5450 3250 5450
@@
 Wire Wire Line
 	800  900  2850 900
-Wire Wire Line
-	4550 4600 4600 4600
-Wire Wire Line
-	4600 4600 4600 4125
-Wire Wire Line
-	4600 4125 1175 4125
-Wire Wire Line
-	1175 4125 1175 4450
-Wire Wire Line
-	1175 4450 1250 4450
 Wire Wire Line
 	750  5450 750  7400
@@
 Wire Notes Line
 	1850 7225 1850 5800
+Wire Wire Line
+	6300 7000 950  7000
+Connection ~ 4650 4450
+Wire Wire Line
+	4650 3950 4650 4450
+Connection ~ 4650 3950
+Wire Bus Line
+	850  4200 850  6900
+Wire Wire Line
+	3250 5800 2950 5800
+Wire Wire Line
+	2950 5800 2950 6900
+Wire Wire Line
+	2950 6900 6200 6900
+Wire Wire Line
+	6200 6900 6200 6250
+Wire Wire Line
+	6200 6250 7300 6250
+Connection ~ 6550 6250
+$Sheet
+S 4800 4350 1300 2350
+U 4DD13EAC
+F0 "CTT/PS3" 60
+F1 "ctt_ps/ctt_ps3.sch" 60
+F2 "DO0" I R 6100 4450 60
+F3 "DO1" I R 6100 4550 60
+F4 "DO2" I R 6100 4650 60
+F5 "DO3" I R 6100 4750 60
+F6 "DO4" I R 6100 4850 60
+F7 "DO5" I R 6100 4950 60
+F8 "DO6" I R 6100 5050 60
+F9 "DO7" I R 6100 5150 60
+F10 "GND" U L 4800 6600 60
+F11 "Um1" O R 6100 6600 60
+F12 "-SL6" I R 6100 5300 60
+F13 "5V 100mA AC" I R 6100 5450 60
+F14 "5V 100mA AC COM" U R 6100 5550 60
+F15 "5V 100mA AC" I R 6100 5650 60
+F16 "+5V" I L 4800 4450 60
+F17 "-NPN/PNP" I R 6100 5800 60
+$EndSheet
 $Comp
 L RELAY J1
@@
 Text Notes 2150 4900 0    60   ~ 0
 CN1
-Text Label 4600 4325 1    60   ~ 0
-78
-Text Label 1175 4450 1    60   ~ 0
-78
 Text Label 1120 5050 0    60   ~ 0
 27
@@
 Entry Wire Line
 	6600 5450 6700 5550
-Text Notes 4100 4640 0    60   ~ 0
-CN1
-Text Notes 3600 5330 0    60   ~ 0
-CN1
-Text Notes 4090 5580 0    60   ~ 0
-CN2
-Text Notes 3830 6610 0    60   ~ 0
-CN2
 Text Label 3100 5650 2    60   ~ 0
 72
@@
 F9 "DO7" I L 3250 5150 60
 F10 "GND" U R 4550 6600 60
-F11 "+Um3" O L 3250 6600 60
-F12 "-Um3" O L 3250 6500 60
-F13 "-SL7" I L 3250 5300 60
-F14 "OVL" O R 4550 4600 60
-F15 "25V 1A AC COM" U L 3250 5550 60
-F16 "25V 1A AC" I L 3250 5450 60
-F17 "25V 1A AC" I L 3250 5650 60
-F18 "+15V" O R 4550 4750 60
+F11 "Um3" O L 3250 6600 60
+F12 "-SL7" I L 3250 5300 60
+F13 "25V 1A AC COM" U L 3250 5550 60
+F14 "25V 1A AC" I L 3250 5450 60
+F15 "25V 1A AC" I L 3250 5650 60
+F16 "+5V" I R 4550 4450 60
+F17 "-NPN/PNP" I L 3250 5800 60
 $EndSheet
 Text Label 2600 800  0    60   ~ 0
@@
 Entry Wire Line
 	2850 800  2950 900
-Text Label 1200 6075 0    60   ~ 0
+Text Label 1200 6050 0    60   ~ 0
 77
-Text Label 1200 5825 0    60   ~ 0
+Text Label 1200 5875 0    60   ~ 0
 76
 Text Label 8800 5750 0    60   ~ 0
@@
 Text Label 1200 5675 0    60   ~ 0
 27
-Text Label 1200 6225 0    60   ~ 0
+Text Label 1200 6250 0    60   ~ 0
 31
-Text Label 1000 7100 0    60   ~ 0
+Text Label 1000 7000 0    60   ~ 0
 30
-Text Label 1000 6750 0    60   ~ 0
+Text Label 1000 6600 0    60   ~ 0
 29
-Text Label 2400 7025 0    60   ~ 0
-62
-Text Label 2400 7175 0    60   ~ 0
-63
-Text Label 6200 6850 1    60   ~ 0
-63
-Text Label 6200 6500 0    60   ~ 0
-62
-Text Label 2400 6825 0    60   ~ 0
-61
-Text Label 2400 6675 0    60   ~ 0
-60
-Text Label 3050 6600 0    60   ~ 0
-61
-Text Label 3050 6500 0    60   ~ 0
-60
-Text Label 2400 5750 0    60   ~ 0
+Text Label 2425 5775 0    60   ~ 0
 59
 Text Label 2400 6150 0    60   ~ 0
@@
 Text Label 7100 6500 0    60   ~ 0
 58
-Text Label 2400 7500 0    60   ~ 0
+Text Label 2150 7400 0    60   ~ 0
 33
 Text Label 7100 6350 0    60   ~ 0
@@
 Entry Wire Line
 	2850 1750 2950 1650
-Text Notes 5550 4850 0    60   ~ 0
-CN1
-Text Notes 3600 4850 0    60   ~ 0
-CN1
 Text Notes 7700 6600 0    60   ~ 0
 CN3
@@
 	6350 3100 6450 3200
 Entry Wire Line
-	850  6125 950  6225
+	850  6150 950  6250
 Entry Wire Line
 	850  5575 950  5675
 Entry Wire Line
-	850  6650 950  6750
-Entry Wire Line
-	850  7000 950  7100
+	850  6500 950  6600
+Entry Wire Line
+	850  6900 950  7000
 Entry Wire Line
 	6350 3400 6450 3500
@@
 L SWITCH_INV JC1
 U 1 1 4DD13F71
-P 1850 5750
-F 0 "JC1" H 1600 5600 50  0000 C CNN
-F 1 "SWITCH_INV" H 1700 5600 50  0001 C CNN
-	1    1850 5750
+P 1875 5775
+F 0 "JC1" H 1625 5625 50  0000 C CNN
+F 1 "SWITCH_INV" H 1725 5625 50  0001 C CNN
+	1    1875 5775
 	-1   0    0    1
 $EndComp
@@
 L SWITCH_INV JC2
 U 1 1 4DD13ED3
-P 1850 6150
-F 0 "JC2" H 1600 6300 50  0000 C CNN
-F 1 "SWITCH_INV" H 1700 6000 50  0001 C CNN
-	1    1850 6150
+P 1875 6150
+F 0 "JC2" H 1625 6300 50  0000 C CNN
+F 1 "SWITCH_INV" H 1725 6000 50  0001 C CNN
+	1    1875 6150
 	-1   0    0    -1
-$EndComp
-$Comp
-L SWITCH_INV JC4
-U 1 1 4DD13ED0
-P 1850 7100
-F 0 "JC4" H 1600 6950 50  0000 C CNN
-F 1 "SWITCH_INV" H 1700 6950 50  0001 C CNN
-	1    1850 7100
-	1    0    0    1
-$EndComp
-$Comp
-L SWITCH_INV JC3
-U 1 1 4DD0087F
-P 1850 6750
-F 0 "JC3" H 1600 6600 50  0000 C CNN
-F 1 "SWITCH_INV" H 1700 6600 50  0001 C CNN
-	1    1850 6750
-	1    0    0    1
 $EndComp
 Text Label 7100 6250 0    60   ~ 0
@@
 F14 "POL" O L 7300 6350 60
 $EndSheet
-$Sheet
-S 4800 4350 1300 2350
-U 4DD13EAC
-F0 "CTT/PS3" 60
-F1 "ctt_ps/ctt_ps3.sch" 60
-F2 "DO0" I R 6100 4450 60
-F3 "DO1" I R 6100 4550 60
-F4 "DO2" I R 6100 4650 60
-F5 "DO3" I R 6100 4750 60
-F6 "DO4" I R 6100 4850 60
-F7 "DO5" I R 6100 4950 60
-F8 "DO6" I R 6100 5050 60
-F9 "DO7" I R 6100 5150 60
-F10 "GND" U L 4800 6600 60
-F11 "-Um1" O R 6100 6500 60
-F12 "+Um1" O R 6100 6600 60
-F13 "-SL6" I R 6100 5300 60
-F14 "5V 100mA AC" I R 6100 5450 60
-F15 "5V 100mA AC COM" U R 6100 5550 60
-F16 "5V 100mA AC" I R 6100 5650 60
-F17 "+15V" I L 4800 4750 60
-$EndSheet
 Text Notes 4000 3440 0    60   ~ 0

Commit message: 2012.01.08. 2. feltöltés.
Changed lines of the file:
@@
-EESchema Schematic File Version 2  date 2012.01.08. 14:43:31
+EESchema Schematic File Version 2  date 2012.01.08. 16:55:02
 LIBS:power
 LIBS:device
@@
 Comment4 ""
 $EndDescr
+Text Label 3000 6600 0    60   ~ 0
+29
+Text Label 3000 5800 0    60   ~ 0
+32
+Text Label 6200 5800 0    60   ~ 0
+32
 Connection ~ 6550 5800
 Wire Wire Line
