File: cad_files/ctt_sw/ctt_sw2.kicad_pcb (KiCad board)
At the start: 2 copper layers, 141 x 73.7 mm, 76 parts, among them J1 Reed_relay, J10 Reed_relay, J11 Reed_relay, J12 Reed_relay, J2 Reed_relay, J2-2 Reed_relay, J3 Reed_relay, J4 Reed_relay, J5 Reed_relay, J6 Reed_relay, J7 Reed_relay, J8 Reed_relay, J8-2 Reed_relay, J9 Reed_relay

Commit message: 220905
Parts:
- renumbered J1 to K1, J10 to K10, JC10 to K10a, J11 to K11, JC11 to K11a, J12 to K12, JC12 to K12a, JC1 to K1a, J2 to K2, J2-2 to K2-2, JC2-2 to K2-2a, JC2 to K2a, J3 to K3, JC3 to K3a, J4 to K4, JC4 to K4a, J5 to K5, JC5 to K5a, J6 to K6, JC6 to K6a, J7 to K7, JC7 to K7a, J8 to K8, J8-2 to K8-2, JC8-2 to K8-2a, JC8 to K8a, J9 to K9, JC9 to K9a
Changed lines of the file:
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@@
     (visible_elements 7FFFFFFF)
     (pcbplotparams
-      (layerselection 0x00000_80000000)
+      (layerselection 0x00020_00000000)
       (usegerberextensions false)
       (excludeedgelayer false)
       (linewidth 0.100000)
-      (plotframeref true)
+      (plotframeref false)
       (viasonmask false)
       (mode 1)
@@
       (psnegative false)
       (psa4output false)
-      (plotreference true)
+      (plotreference false)
       (plotvalue false)
       (plotinvisibletext false)
-      (padsonsilk true)
+      (padsonsilk false)
       (subtractmaskfromsilk false)
-      (outputformat 4)
-      (mirror true)
-      (drillshape 1)
+      (outputformat 1)
+      (mirror false)
+      (drillshape 0)
       (scaleselection 1)
       (outputdirectory ""))
@@
     (tags R)
     (autoplace_cost180 10)
-    (fp_text reference JC12 (at 0.635 0) (layer F.SilkS)
+    (fp_text reference K12a (at 0.635 0) (layer F.SilkS)
       (effects (font (size 1.397 1.27) (thickness 0.2032)))
     )
@@
     (tags R)
     (autoplace_cost180 10)
-    (fp_text reference JC11 (at 0 0 180) (layer F.SilkS)
+    (fp_text reference K11a (at 0 0 180) (layer F.SilkS)
       (effects (font (size 1.397 1.27) (thickness 0.2032)))
     )
@@
     (tags R)
     (autoplace_cost180 10)
-    (fp_text reference JC10 (at 0 0) (layer F.SilkS)
+    (fp_text reference K10a (at 0 0) (layer F.SilkS)
       (effects (font (size 1.397 1.27) (thickness 0.2032)))
     )
@@
     (tags R)
     (autoplace_cost180 10)
-    (fp_text reference JC9 (at 0 0 180) (layer F.SilkS)
+    (fp_text reference K9a (at 0 0 180) (layer F.SilkS)
       (effects (font (size 1.397 1.27) (thickness 0.2032)))
     )
@@
     (tags R)
     (autoplace_cost180 10)
-    (fp_text reference JC8-2 (at 0.635 0) (layer F.SilkS)
+    (fp_text reference K8-2a (at 0.635 0) (layer F.SilkS)
       (effects (font (size 1.397 1.27) (thickness 0.2032)))
     )
@@
     (tags R)
     (autoplace_cost180 10)
-    (fp_text reference JC8 (at 0 0 180) (layer F.SilkS)
+    (fp_text reference K8a (at 0 0 180) (layer F.SilkS)
       (effects (font (size 1.397 1.27) (thickness 0.2032)))
     )
@@
     (tags R)
     (autoplace_cost180 10)
-    (fp_text reference JC7 (at 0 0) (layer F.SilkS)
+    (fp_text reference K7a (at 0 0) (layer F.SilkS)
       (effects (font (size 1.397 1.27) (thickness 0.2032)))
     )
@@
     (tags R)
     (autoplace_cost180 10)
-    (fp_text reference JC6 (at 0 0 180) (layer F.SilkS)
+    (fp_text reference K6a (at 0 0 180) (layer F.SilkS)
       (effects (font (size 1.397 1.27) (thickness 0.2032)))
     )
@@
     (tags R)
     (autoplace_cost180 10)
-    (fp_text reference JC5 (at 0 0) (layer F.SilkS)
+    (fp_text reference K5a (at 0 0) (layer F.SilkS)
       (effects (font (size 1.397 1.27) (thickness 0.2032)))
     )
@@
     (tags R)
     (autoplace_cost180 10)
-    (fp_text reference JC4 (at 0 0 180) (layer F.SilkS)
+    (fp_text reference K4a (at 0 0 180) (layer F.SilkS)
       (effects (font (size 1.397 1.27) (thickness 0.2032)))
     )
@@
     (tags R)
     (autoplace_cost180 10)
-    (fp_text reference JC3 (at 0 0) (layer F.SilkS)
+    (fp_text reference K3a (at 0 0) (layer F.SilkS)
       (effects (font (size 1.397 1.27) (thickness 0.2032)))
     )
@@
     (tags R)
     (autoplace_cost180 10)
-    (fp_text reference JC2-2 (at 0 0) (layer F.SilkS)
+    (fp_text reference K2-2a (at 0 0) (layer F.SilkS)
       (effects (font (size 1.397 1.27) (thickness 0.2032)))
     )
@@
     (tags R)
     (autoplace_cost180 10)
-    (fp_text reference JC2 (at 0 0) (layer F.SilkS)
+    (fp_text reference K2a (at 0 0) (layer F.SilkS)
       (effects (font (size 1.397 1.27) (thickness 0.2032)))
     )
@@
     (tags R)
     (autoplace_cost180 10)
-    (fp_text reference JC1 (at 0 0 180) (layer F.SilkS)
+    (fp_text reference K1a (at 0 0 180) (layer F.SilkS)
       (effects (font (size 1.397 1.27) (thickness 0.2032)))
     )
@@
     (descr "Connecteurs 2 pins")
     (tags "CONN DEV")
-    (fp_text reference J12 (at -5.08 0 180) (layer F.SilkS)
+    (fp_text reference K12 (at -5.08 0 180) (layer F.SilkS)
       (effects (font (size 1.72974 1.08712) (thickness 0.3048)))
     )
@@
     (descr "Connecteurs 2 pins")
     (tags "CONN DEV")
-    (fp_text reference J11 (at -5.08 0 180) (layer F.SilkS)
+    (fp_text reference K11 (at -5.08 0 180) (layer F.SilkS)
       (effects (font (size 1.72974 1.08712) (thickness 0.3048)))
     )
@@
     (descr "Connecteurs 2 pins")
     (tags "CONN DEV")
-    (fp_text reference J10 (at -5.08 0 180) (layer F.SilkS)
+    (fp_text reference K10 (at -5.08 0 180) (layer F.SilkS)
       (effects (font (size 1.72974 1.08712) (thickness 0.3048)))
     )
@@
     (descr "Connecteurs 2 pins")
     (tags "CONN DEV")
-    (fp_text reference J9 (at -4.445 0 180) (layer F.SilkS)
+    (fp_text reference K9 (at -4.445 0 180) (layer F.SilkS)
       (effects (font (size 1.72974 1.08712) (thickness 0.3048)))
     )
@@
     (descr "Connecteurs 2 pins")
     (tags "CONN DEV")
-    (fp_text reference J8-2 (at 0 -3.175 180) (layer F.SilkS)
+    (fp_text reference K8-2 (at 0 -3.175 180) (layer F.SilkS)
       (effects (font (size 1.72974 1.08712) (thickness 0.3048)))
     )
@@
     (descr "Connecteurs 2 pins")
     (tags "CONN DEV")
-    (fp_text reference J8 (at -4.445 0 180) (layer F.SilkS)
+    (fp_text reference K8 (at -4.445 0 180) (layer F.SilkS)
       (effects (font (size 1.72974 1.08712) (thickness 0.3048)))
     )
@@
     (descr "Connecteurs 2 pins")
     (tags "CONN DEV")
-    (fp_text reference J7 (at -4.445 0 180) (layer F.SilkS)
+    (fp_text reference K7 (at -4.445 0 180) (layer F.SilkS)
       (effects (font (size 1.72974 1.08712) (thickness 0.3048)))
     )
@@
     (descr "Connecteurs 2 pins")
     (tags "CONN DEV")
-    (fp_text reference J6 (at -4.445 0 180) (layer F.SilkS)
+    (fp_text reference K6 (at -4.445 0 180) (layer F.SilkS)
       (effects (font (size 1.72974 1.08712) (thickness 0.3048)))
     )
@@
     (descr "Connecteurs 2 pins")
     (tags "CONN DEV")
-    (fp_text reference J5 (at -4.445 0 180) (layer F.SilkS)
+    (fp_text reference K5 (at -4.445 0 180) (layer F.SilkS)
       (effects (font (size 1.72974 1.08712) (thickness 0.3048)))
     )
@@
     (descr "Connecteurs 2 pins")
     (tags "CONN DEV")
-    (fp_text reference J4 (at -4.445 0 180) (layer F.SilkS)
+    (fp_text reference K4 (at -4.445 0 180) (layer F.SilkS)
       (effects (font (size 1.72974 1.08712) (thickness 0.3048)))
     )
@@
     (descr "Connecteurs 2 pins")
     (tags "CONN DEV")
-    (fp_text reference J3 (at -4.445 0 180) (layer F.SilkS)
+    (fp_text reference K3 (at -4.445 0 180) (layer F.SilkS)
       (effects (font (size 1.72974 1.08712) (thickness 0.3048)))
     )
@@
     (descr "Connecteurs 2 pins")
     (tags "CONN DEV")
-    (fp_text reference J2-2 (at -5.715 0 180) (layer F.SilkS)
+    (fp_text reference K2-2 (at -5.715 0 180) (layer F.SilkS)
       (effects (font (size 1.72974 1.08712) (thickness 0.3048)))
     )
@@
     (descr "Connecteurs 2 pins")
     (tags "CONN DEV")
-    (fp_text reference J2 (at -4.445 0 180) (layer F.SilkS)
+    (fp_text reference K2 (at -4.445 0 180) (layer F.SilkS)
       (effects (font (size 1.72974 1.08712) (thickness 0.3048)))
     )
@@
     (descr "Connecteurs 2 pins")
     (tags "CONN DEV")
-    (fp_text reference J1 (at -4.445 0 180) (layer F.SilkS)
+    (fp_text reference K1 (at -4.445 0 180) (layer F.SilkS)
       (effects (font (size 1.72974 1.08712) (thickness 0.3048)))
     )
