File: cad_files/ctt_ps/ctt_ps4.sch (KiCad schematic (older format))
At the start: 11 parts, among them SW1a SPST, SW1b SPST

Commit message: 220902
Parts:
- F1: symbol FUSE-EU -> Fuse-EU
Changed lines of the file:
@@
-EESchema Schematic File Version 2  date 2012.01.28. 6:39:46
+EESchema Schematic File Version 2
+LIBS:ctt-rescue
 LIBS:power
 LIBS:device
@@
 LIBS:memory
 LIBS:xilinx
-LIBS:special
 LIBS:microcontrollers
 LIBS:dsp
@@
 LIBS:valves
 LIBS:ctt-cache
-EELAYER 24  0
+EELAYER 25 0
 EELAYER END
-$Descr A4 11700 8267
+$Descr A4 11693 8268
+encoding utf-8
 Sheet 5 11
 Title "CTT Transistor tester - CTT/PS4 power supply unit"
@@
 CN1
 $Comp
-L GND #PWR?
+L GND-RESCUE-ctt #PWR?
 U 1 1 4DD3D9AA
 P 7400 2400
 F 0 "#PWR?" H 7400 2400 30  0001 C CNN
 F 1 "GND" H 7400 2330 30  0001 C CNN
+F 2 "" H 7400 2400 60  0001 C CNN
+F 3 "" H 7400 2400 60  0001 C CNN
 	1    7400 2400
 	1    0    0    -1
@@
 F 0 "SW1b" H 6900 1800 70  0000 C CNN
 F 1 "SPST" H 6900 1850 70  0001 C CNN
+F 2 "" H 6900 1950 60  0001 C CNN
+F 3 "" H 6900 1950 60  0001 C CNN
 	1    6900 1950
 	1    0    0    -1
@@
 F 0 "SW1a" H 6900 1450 70  0000 C CNN
 F 1 "SPST" H 6900 1150 70  0001 C CNN
+F 2 "" H 6900 1250 60  0001 C CNN
+F 3 "" H 6900 1250 60  0001 C CNN
 	1    6900 1250
 	1    0    0    -1
 $EndComp
 $Comp
-L FUSE-EU F1
+L Fuse-EU F1
 U 1 1 4DD2D28B
 P 5950 1250
 F 0 "F1" V 6050 1250 50  0000 C CNN
 F 1 "500 mA T" V 5850 1250 50  0000 C CNN
+F 2 "" H 5950 1250 60  0001 C CNN
+F 3 "" H 5950 1250 60  0001 C CNN
 	1    5950 1250
 	0    1    1    0
@@
 F 0 "S6" V 5150 5700 40  0000 C CNN
 F 1 "INDUCTOR" V 5050 5700 40  0001 C CNN
+F 2 "" H 5250 5700 60  0001 C CNN
+F 3 "" H 5250 5700 60  0001 C CNN
 	1    5250 5700
 	1    0    0    1
@@
 F 0 "S7" V 5150 6400 40  0000 C CNN
 F 1 "INDUCTOR" V 5050 6400 40  0001 C CNN
+F 2 "" H 5250 6400 60  0001 C CNN
+F 3 "" H 5250 6400 60  0001 C CNN
 	1    5250 6400
 	1    0    0    1
@@
 F 0 "S5" V 5150 4850 40  0000 C CNN
 F 1 "INDUCTOR" V 5050 4850 40  0001 C CNN
+F 2 "" H 5250 4850 60  0001 C CNN
+F 3 "" H 5250 4850 60  0001 C CNN
 	1    5250 4850
 	1    0    0    1
@@
 F 0 "S4" V 5150 4150 40  0000 C CNN
 F 1 "INDUCTOR" V 5050 4150 40  0001 C CNN
+F 2 "" H 5250 4150 60  0001 C CNN
+F 3 "" H 5250 4150 60  0001 C CNN
 	1    5250 4150
 	1    0    0    1
@@
 F 0 "S3" V 5150 3300 40  0000 C CNN
 F 1 "INDUCTOR" V 5050 3300 40  0001 C CNN
+F 2 "" H 5250 3300 60  0001 C CNN
+F 3 "" H 5250 3300 60  0001 C CNN
 	1    5250 3300
 	1    0    0    1
@@
 F 0 "S2" V 5150 2450 40  0000 C CNN
 F 1 "INDUCTOR" V 5050 2450 40  0001 C CNN
+F 2 "" H 5250 2450 60  0001 C CNN
+F 3 "" H 5250 2450 60  0001 C CNN
 	1    5250 2450
 	1    0    0    1
@@
 F 0 "P" V 5350 1600 40  0000 C CNN
 F 1 "INDUCTOR" V 5300 1600 40  0001 C CNN
+F 2 "" H 5450 1600 60  0001 C CNN
+F 3 "" H 5450 1600 60  0001 C CNN
 	1    5450 1600
 	-1   0    0    1
@@
 F 0 "S1" V 5150 1600 40  0000 C CNN
 F 1 "INDUCTOR" V 5050 1600 40  0001 C CNN
+F 2 "" H 5250 1600 60  0001 C CNN
+F 3 "" H 5250 1600 60  0001 C CNN
 	1    5250 1600
 	1    0    0    1

Commit message: 220903
Changed lines of the file:
@@
 $Descr A4 11693 8268
 encoding utf-8
-Sheet 5 11
+Sheet 10 11
 Title "CTT Transistor tester - CTT/PS4 power supply unit"
 Date "28 jan 2012"
@@
 U 1 1 4DD2D2D7
 P 6900 1950
-F 0 "SW1b" H 6900 1800 70  0000 C CNN
+F 0 "SW1b" H 6900 1800 50  0000 C CNN
 F 1 "SPST" H 6900 1850 70  0001 C CNN
 F 2 "" H 6900 1950 60  0001 C CNN
@@
 U 1 1 4DD2D2CB
 P 6900 1250
-F 0 "SW1a" H 6900 1450 70  0000 C CNN
+F 0 "SW1a" H 6900 1450 50  0000 C CNN
 F 1 "SPST" H 6900 1150 70  0001 C CNN
 F 2 "" H 6900 1250 60  0001 C CNN
@@
 F 3 "" H 5950 1250 60  0001 C CNN
 	1    5950 1250
-	0    1    1    0
+	0    1    -1   0
 $EndComp
-Text Notes 5275 1125 0    60   ~ 0
+Text Notes 5275 1125 0    50   ~ 0
 Tr1
 Text Notes 5075 6750 0    60   ~ 0

Commit message: 220910
Changed lines of the file:
@@
 $EndDescr
 Wire Wire Line
-	6450 1950 5450 1950
+	6500 1950 5450 1950
 Wire Wire Line
-	7400 2400 7400 1600
+	7400 1600 7400 2400
 Wire Notes Line
-	6900 1250 6900 1850
+	6750 1250 6750 1850
 Wire Wire Line
-	7600 1950 7350 1950
+	7600 1950 7000 1950
 Wire Wire Line
 	5700 1250 5450 1250
@@
 	5250 3800 4750 3800
 Wire Wire Line
-	5250 4550 5250 4450
+	5250 4450 5250 4550
 Wire Wire Line
 	4750 4500 5250 4500
@@
 	5450 1950 5450 1900
 Wire Wire Line
-	7350 1250 7600 1250
+	7000 1250 7600 1250
 Wire Wire Line
 	4750 6900 5800 6900
@@
 Connection ~ 7400 2250
 Wire Wire Line
-	6450 1250 6200 1250
+	6500 1250 6200 1250
 Text Notes 7450 1950 0    60   ~ 0
 3
@@
 L SPST SW1b
 U 1 1 4DD2D2D7
-P 6900 1950
-F 0 "SW1b" H 6900 1800 50  0000 C CNN
-F 1 "SPST" H 6900 1850 70  0001 C CNN
-F 2 "" H 6900 1950 60  0001 C CNN
-F 3 "" H 6900 1950 60  0001 C CNN
-	1    6900 1950
+P 6750 1950
+F 0 "SW1b" H 6750 1800 50  0000 C CNN
+F 1 "SPST" H 6750 1850 70  0001 C CNN
+F 2 "" H 6750 1950 60  0001 C CNN
+F 3 "" H 6750 1950 60  0001 C CNN
+	1    6750 1950
 	1    0    0    -1
 $EndComp
@@
 L SPST SW1a
 U 1 1 4DD2D2CB
-P 6900 1250
-F 0 "SW1a" H 6900 1450 50  0000 C CNN
-F 1 "SPST" H 6900 1150 70  0001 C CNN
-F 2 "" H 6900 1250 60  0001 C CNN
-F 3 "" H 6900 1250 60  0001 C CNN
-	1    6900 1250
+P 6750 1250
+F 0 "SW1a" H 6750 1450 50  0000 C CNN
+F 1 "SPST" H 6750 1150 70  0001 C CNN
+F 2 "" H 6750 1250 60  0001 C CNN
+F 3 "" H 6750 1250 60  0001 C CNN
+	1    6750 1250
 	1    0    0    -1
 $EndComp
