File: cad_files/ctt_ps/ctt_ps1.sch (KiCad schematic (older format))
At the start: 38 parts, among them IC1 7905, IC2 78S05, T1 BC182, T2 BC301

Commit message: 220902
Parts:
- C15: symbol CP -> CP-RESCUE-ctt
- C2, C3, C6, C7: symbol C -> C-RESCUE-ctt
- R1: symbol R -> R-RESCUE-ctt
Changed lines of the file:
@@
-EESchema Schematic File Version 2  date 2012.01.28. 6:39:46
+EESchema Schematic File Version 2
+LIBS:ctt-rescue
 LIBS:power
 LIBS:device
@@
 LIBS:memory
 LIBS:xilinx
-LIBS:special
 LIBS:microcontrollers
 LIBS:dsp
@@
 LIBS:valves
 LIBS:ctt-cache
-EELAYER 24  0
+EELAYER 25 0
 EELAYER END
-$Descr A4 11700 8267
+$Descr A4 11693 8268
+encoding utf-8
 Sheet 7 11
 Title "CTT Transistor tester - CTT/PS1 power supply unit"
@@
 CN4
 $Comp
-L CP C15
+L CP-RESCUE-ctt C15
 U 1 1 4DDD087E
 P 4200 5100
 F 0 "C15" H 4150 4700 50  0000 L CNN
 F 1 "22u 200V" H 4350 5100 50  0000 L CNN
+F 2 "" H 4200 5100 60  0001 C CNN
+F 3 "" H 4200 5100 60  0001 C CNN
 	1    4200 5100
 	1    0    0    -1
@@
 F 0 "D17" H 4850 4600 40  0000 C CNN
 F 1 "1N4001" H 4600 4450 40  0000 C CNN
+F 2 "" H 4700 4550 60  0001 C CNN
+F 3 "" H 4700 4550 60  0001 C CNN
 	1    4700 4550
 	0    -1   -1   0
@@
 F 0 "D18" H 4050 4600 40  0000 C CNN
 F 1 "1N4001" H 4300 4450 40  0000 C CNN
+F 2 "" H 4200 4550 60  0001 C CNN
+F 3 "" H 4200 4550 60  0001 C CNN
 	1    4200 4550
 	0    -1   1    0
@@
 F 0 "C14" H 4475 4925 50  0000 L CNN
 F 1 "10u" H 4275 4675 50  0000 L CNN
+F 2 "" H 4450 4800 60  0001 C CNN
+F 3 "" H 4450 4800 60  0001 C CNN
 	1    4450 4800
 	0    -1   1    0
@@
 F 0 "D15" H 5850 4600 40  0000 C CNN
 F 1 "1N4001" H 5600 4450 40  0000 C CNN
+F 2 "" H 5700 4550 60  0001 C CNN
+F 3 "" H 5700 4550 60  0001 C CNN
 	1    5700 4550
 	0    -1   -1   0
@@
 F 0 "D16" H 5050 4600 40  0000 C CNN
 F 1 "1N4001" H 5300 4450 40  0000 C CNN
+F 2 "" H 5200 4550 60  0001 C CNN
+F 3 "" H 5200 4550 60  0001 C CNN
 	1    5200 4550
 	0    -1   1    0
@@
 F 0 "C12" H 5475 4925 50  0000 L CNN
 F 1 "10u" H 5275 4675 50  0000 L CNN
+F 2 "" H 5450 4800 60  0001 C CNN
+F 3 "" H 5450 4800 60  0001 C CNN
 	1    5450 4800
 	0    -1   1    0
@@
 F 0 "C13" H 4975 4425 50  0000 L CNN
 F 1 "10u" H 4775 4175 50  0000 L CNN
+F 2 "" H 4950 4300 60  0001 C CNN
+F 3 "" H 4950 4300 60  0001 C CNN
 	1    4950 4300
 	0    -1   1    0
@@
 F 0 "C11" H 5975 4425 50  0000 L CNN
 F 1 "10u" H 5775 4175 50  0000 L CNN
+F 2 "" H 5950 4300 60  0001 C CNN
+F 3 "" H 5950 4300 60  0001 C CNN
 	1    5950 4300
 	0    -1   1    0
@@
 F 0 "C10" H 6475 4925 50  0000 L CNN
 F 1 "10u" H 6275 4675 50  0000 L CNN
+F 2 "" H 6450 4800 60  0001 C CNN
+F 3 "" H 6450 4800 60  0001 C CNN
 	1    6450 4800
 	0    -1   1    0
@@
 F 0 "C9" H 6975 4425 50  0000 L CNN
 F 1 "10u" H 6775 4175 50  0000 L CNN
+F 2 "" H 6950 4300 60  0001 C CNN
+F 3 "" H 6950 4300 60  0001 C CNN
 	1    6950 4300
 	0    -1   1    0
@@
 F 0 "D14" H 6050 4600 40  0000 C CNN
 F 1 "1N4001" H 6300 4450 40  0000 C CNN
+F 2 "" H 6200 4550 60  0001 C CNN
+F 3 "" H 6200 4550 60  0001 C CNN
 	1    6200 4550
 	0    -1   1    0
@@
 F 0 "D13" H 6850 4600 40  0000 C CNN
 F 1 "1N4001" H 6600 4450 40  0000 C CNN
+F 2 "" H 6700 4550 60  0001 C CNN
+F 3 "" H 6700 4550 60  0001 C CNN
 	1    6700 4550
 	0    -1   -1   0
@@
 GND
 $Comp
-L C C7
+L C-RESCUE-ctt C7
 U 1 1 4DD3E626
 P 5050 3600
 F 0 "C7" H 5100 3700 50  0000 L CNN
 F 1 "1n" H 4900 3450 50  0000 L CNN
+F 2 "" H 5050 3600 60  0001 C CNN
+F 3 "" H 5050 3600 60  0001 C CNN
 	1    5050 3600
 	1    0    0    -1
 $EndComp
 $Comp
-L C C6
+L C-RESCUE-ctt C6
 U 1 1 4DD3E625
 P 6050 3600
 F 0 "C6" H 5900 3700 50  0000 L CNN
 F 1 "1n" H 6100 3450 50  0000 L CNN
+F 2 "" H 6050 3600 60  0001 C CNN
+F 3 "" H 6050 3600 60  0001 C CNN
 	1    6050 3600
 	1    0    0    -1
@@
 F 0 "C5" H 6500 3700 50  0000 L CNN
 F 1 "1000u 16V" H 6200 3250 50  0000 L CNN
+F 2 "" H 6400 3600 60  0001 C CNN
+F 3 "" H 6400 3600 60  0001 C CNN
 	1    6400 3600
 	-1   0    0    -1
@@
 F 0 "C8" H 4300 3700 50  0000 L CNN
 F 1 "1u" H 4550 3450 50  0000 L CNN
+F 2 "" H 4450 3600 60  0001 C CNN
+F 3 "" H 4450 3600 60  0001 C CNN
 	1    4450 3600
 	-1   0    0    -1
@@
 F 0 "D8" H 7100 3700 40  0000 C CNN
 F 1 "1N4001" H 6750 3550 40  0001 C CNN
+F 2 "" H 6950 3650 60  0001 C CNN
+F 3 "" H 6950 3650 60  0001 C CNN
 	1    6950 3650
 	-1   0    0    -1
@@
 F 0 "D10" H 6800 3750 40  0000 C CNN
 F 1 "1N4001" H 7150 3600 40  0001 C CNN
+F 2 "" H 6950 3800 60  0001 C CNN
+F 3 "" H 6950 3800 60  0001 C CNN
 	1    6950 3800
 	1    0    0    1
@@
 F 0 "D7" H 7100 3400 40  0000 C CNN
 F 1 "BY399" H 6950 2750 40  0000 C CNN
+F 2 "" H 6950 3350 60  0001 C CNN
+F 3 "" H 6950 3350 60  0001 C CNN
 	1    6950 3350
 	-1   0    0    -1
@@
 F 0 "D9" H 6800 3450 40  0000 C CNN
 F 1 "1N4001" H 6950 3200 40  0001 C CNN
+F 2 "" H 6950 3500 60  0001 C CNN
+F 3 "" H 6950 3500 60  0001 C CNN
 	1    6950 3500
 	1    0    0    1
@@
 F 0 "D11" H 5450 3050 40  0000 C CNN
 F 1 "BY399" H 5750 2900 40  0000 C CNN
+F 2 "" H 5550 2950 60  0001 C CNN
+F 3 "" H 5550 2950 60  0001 C CNN
 	1    5550 2950
 	1    0    0    1
@@
 F 0 "D12" H 4850 3700 40  0000 C CNN
 F 1 "BY399" V 4400 3600 40  0000 C CNN
+F 2 "" H 4750 3600 60  0001 C CNN
+F 3 "" H 4750 3600 60  0001 C CNN
 	1    4750 3600
 	0    1    -1   0
@@
 F 0 "IC1" H 5550 2350 60  0000 C CNN
 F 1 "7905" H 5550 1550 60  0000 C CNN
+F 2 "" H 5550 2150 60  0001 C CNN
+F 3 "" H 5550 2150 60  0001 C CNN
 	1    5550 2150
 	1    0    0    -1
@@
 F 0 "D6" H 4650 2500 40  0000 C CNN
 F 1 "1N4001" V 5100 2400 40  0000 C CNN
+F 2 "" H 4750 2400 60  0001 C CNN
+F 3 "" H 4750 2400 60  0001 C CNN
 	1    4750 2400
 	0    1    1    0
@@
 P 5550 1750
 F 0 "D5" H 5650 1850 40  0000 C CNN
-F 1 "1N4001" H 5350 1700 40  0000 C CNN
+F 1 "1N4001" H 5350 1700 50  0000 C CNN
+F 2 "" H 5550 1750 60  0001 C CNN
+F 3 "" H 5550 1750 60  0001 C CNN
 	1    5550 1750
 	-1   0    0    1
@@
 F 0 "D3" H 6800 2250 40  0000 C CNN
 F 1 "1N4001" H 6950 2000 40  0001 C CNN
+F 2 "" H 6950 2300 60  0001 C CNN
+F 3 "" H 6950 2300 60  0001 C CNN
 	1    6950 2300
 	-1   0    0    1
@@
 F 0 "D1" H 7100 2200 40  0000 C CNN
 F 1 "1N4001" H 6950 1550 40  0000 C CNN
+F 2 "" H 6950 2150 60  0001 C CNN
+F 3 "" H 6950 2150 60  0001 C CNN
 	1    6950 2150
 	1    0    0    -1
@@
 F 0 "D4" H 6800 2550 40  0000 C CNN
 F 1 "1N4001" H 7150 2400 40  0001 C CNN
+F 2 "" H 6950 2600 60  0001 C CNN
+F 3 "" H 6950 2600 60  0001 C CNN
 	1    6950 2600
 	-1   0    0    1
@@
 F 0 "D2" H 7100 2500 40  0000 C CNN
 F 1 "1N4001" H 6750 2350 40  0001 C CNN
+F 2 "" H 6950 2450 60  0001 C CNN
+F 3 "" H 6950 2450 60  0001 C CNN
 	1    6950 2450
 	1    0    0    -1
@@
 F 0 "C4" H 4300 2300 50  0000 L CNN
 F 1 "1u" H 4550 2550 50  0000 L CNN
+F 2 "" H 4450 2400 60  0001 C CNN
+F 3 "" H 4450 2400 60  0001 C CNN
 	1    4450 2400
 	-1   0    0    1
@@
 F 0 "C1" H 6450 2300 50  0000 L CNN
 F 1 "220u 16V" H 6250 2750 50  0000 L CNN
+F 2 "" H 6400 2400 60  0001 C CNN
+F 3 "" H 6400 2400 60  0001 C CNN
 	1    6400 2400
 	-1   0    0    1
 $EndComp
 $Comp
-L C C2
+L C-RESCUE-ctt C2
 U 1 1 4DD3E1DA
 P 6050 2400
 F 0 "C2" H 5900 2500 50  0000 L CNN
 F 1 "1n" H 6100 2250 50  0000 L CNN
+F 2 "" H 6050 2400 60  0001 C CNN
+F 3 "" H 6050 2400 60  0001 C CNN
 	1    6050 2400
 	1    0    0    -1
 $EndComp
 $Comp
-L C C3
+L C-RESCUE-ctt C3
 U 1 1 4DD3E1C5
 P 5050 2400
 F 0 "C3" H 5100 2500 50  0000 L CNN
 F 1 "1n" H 4900 2250 50  0000 L CNN
+F 2 "" H 5050 2400 60  0001 C CNN
+F 3 "" H 5050 2400 60  0001 C CNN
 	1    5050 2400
 	1    0    0    -1
 $EndComp
 $Comp
-L R R1
+L R-RESCUE-ctt R1
 U 1 1 4DD3E1B5
 P 6000 6150
 F 0 "R1" V 5875 6075 50  0000 C CNN
 F 1 "470" V 6125 6200 50  0000 C CNN
+F 2 "" H 6000 6150 60  0001 C CNN
+F 3 "" H 6000 6150 60  0001 C CNN
 	1    6000 6150
 	0    1    1    0
@@
 F 0 "IC2" H 5550 3550 60  0000 C CNN
 F 1 "78S05" H 5550 2750 60  0000 C CNN
+F 2 "" H 5550 3350 60  0001 C CNN
+F 3 "" H 5550 3350 60  0001 C CNN
 	1    5550 3350
 	1    0    0    -1
@@
 F 0 "T1" H 5425 5975 50  0000 R CNN
 F 1 "BC182" H 5650 6450 50  0000 R CNN
+F 2 "" H 5450 6150 60  0001 C CNN
+F 3 "" H 5450 6150 60  0001 C CNN
 	1    5450 6150
 	-1   0    0    -1
@@
 F 0 "T2" H 5075 6225 50  0000 R CNN
 F 1 "BC301" H 5300 6950 50  0000 R CNN
+F 2 "" H 5100 6400 60  0001 C CNN
+F 3 "" H 5100 6400 60  0001 C CNN
 	1    5100 6400
 	-1   0    0    -1

Commit message: 220903
Changed lines of the file:
@@
 $Descr A4 11693 8268
 encoding utf-8
-Sheet 7 11
+Sheet 11 11
 Title "CTT Transistor tester - CTT/PS1 power supply unit"
 Date "28 jan 2012"
@@
 U 1 1 4DD56AE6
 P 4700 4550
-F 0 "D17" H 4850 4600 40  0000 C CNN
-F 1 "1N4001" H 4600 4450 40  0000 C CNN
+F 0 "D17" V 5050 4550 50  0000 C CNN
+F 1 "1N4001" H 4700 4450 50  0000 C CNN
 F 2 "" H 4700 4550 60  0001 C CNN
 F 3 "" H 4700 4550 60  0001 C CNN
@@
 U 1 1 4DD56AE5
 P 4200 4550
-F 0 "D18" H 4050 4600 40  0000 C CNN
-F 1 "1N4001" H 4300 4450 40  0000 C CNN
+F 0 "D18" V 3850 4550 50  0000 C CNN
+F 1 "1N4001" H 4200 4450 50  0000 C CNN
 F 2 "" H 4200 4550 60  0001 C CNN
 F 3 "" H 4200 4550 60  0001 C CNN
@@
 U 1 1 4DD56ADB
 P 5700 4550
-F 0 "D15" H 5850 4600 40  0000 C CNN
-F 1 "1N4001" H 5600 4450 40  0000 C CNN
+F 0 "D15" V 6050 4550 50  0000 C CNN
+F 1 "1N4001" H 5700 4450 50  0000 C CNN
 F 2 "" H 5700 4550 60  0001 C CNN
 F 3 "" H 5700 4550 60  0001 C CNN
@@
 U 1 1 4DD56ADA
 P 5200 4550
-F 0 "D16" H 5050 4600 40  0000 C CNN
-F 1 "1N4001" H 5300 4450 40  0000 C CNN
+F 0 "D16" V 4850 4550 50  0000 C CNN
+F 1 "1N4001" H 5200 4450 50  0000 C CNN
 F 2 "" H 5200 4550 60  0001 C CNN
 F 3 "" H 5200 4550 60  0001 C CNN
@@
 U 1 1 4DD56AD8
 P 4950 4300
-F 0 "C13" H 4975 4425 50  0000 L CNN
-F 1 "10u" H 4775 4175 50  0000 L CNN
+F 0 "C13" V 5150 4250 50  0000 L CNN
+F 1 "10u" V 4750 4250 50  0000 L CNN
 F 2 "" H 4950 4300 60  0001 C CNN
 F 3 "" H 4950 4300 60  0001 C CNN
@@
 U 1 1 4DD3EBAD
 P 5950 4300
-F 0 "C11" H 5975 4425 50  0000 L CNN
-F 1 "10u" H 5775 4175 50  0000 L CNN
+F 0 "C11" V 6150 4250 50  0000 L CNN
+F 1 "10u" V 5750 4250 50  0000 L CNN
 F 2 "" H 5950 4300 60  0001 C CNN
 F 3 "" H 5950 4300 60  0001 C CNN
@@
 U 1 1 4DD3EAF2
 P 6950 4300
-F 0 "C9" H 6975 4425 50  0000 L CNN
-F 1 "10u" H 6775 4175 50  0000 L CNN
+F 0 "C9" V 7150 4250 50  0000 L CNN
+F 1 "10u" V 6750 4250 50  0000 L CNN
 F 2 "" H 6950 4300 60  0001 C CNN
 F 3 "" H 6950 4300 60  0001 C CNN
@@
 U 1 1 4DD3EAD7
 P 6200 4550
-F 0 "D14" H 6050 4600 40  0000 C CNN
-F 1 "1N4001" H 6300 4450 40  0000 C CNN
+F 0 "D14" V 5850 4550 50  0000 C CNN
+F 1 "1N4001" H 6200 4450 50  0000 C CNN
 F 2 "" H 6200 4550 60  0001 C CNN
 F 3 "" H 6200 4550 60  0001 C CNN
@@
 U 1 1 4DD3EAC3
 P 6700 4550
-F 0 "D13" H 6850 4600 40  0000 C CNN
-F 1 "1N4001" H 6600 4450 40  0000 C CNN
+F 0 "D13" V 7050 4550 50  0000 C CNN
+F 1 "1N4001" H 6700 4450 50  0000 C CNN
 F 2 "" H 6700 4550 60  0001 C CNN
 F 3 "" H 6700 4550 60  0001 C CNN
@@
 U 1 1 4DD3E622
 P 6950 3650
-F 0 "D8" H 7100 3700 40  0000 C CNN
+F 0 "D8" H 7100 3700 50  0000 C CNN
 F 1 "1N4001" H 6750 3550 40  0001 C CNN
 F 2 "" H 6950 3650 60  0001 C CNN
@@
 U 1 1 4DD3E621
 P 6950 3800
-F 0 "D10" H 6800 3750 40  0000 C CNN
+F 0 "D10" H 6800 3750 50  0000 C CNN
 F 1 "1N4001" H 7150 3600 40  0001 C CNN
 F 2 "" H 6950 3800 60  0001 C CNN
@@
 U 1 1 4DD3E620
 P 6950 3350
-F 0 "D7" H 7100 3400 40  0000 C CNN
-F 1 "BY399" H 6950 2750 40  0000 C CNN
+F 0 "D7" H 7100 3400 50  0000 C CNN
+F 1 "BY399" H 6950 2750 50  0000 C CNN
 F 2 "" H 6950 3350 60  0001 C CNN
 F 3 "" H 6950 3350 60  0001 C CNN
@@
 U 1 1 4DD3E61F
 P 6950 3500
-F 0 "D9" H 6800 3450 40  0000 C CNN
+F 0 "D9" H 6800 3450 50  0000 C CNN
 F 1 "1N4001" H 6950 3200 40  0001 C CNN
 F 2 "" H 6950 3500 60  0001 C CNN
@@
 U 1 1 4DD3E61E
 P 5550 2950
-F 0 "D11" H 5450 3050 40  0000 C CNN
-F 1 "BY399" H 5750 2900 40  0000 C CNN
+F 0 "D11" H 5450 3050 50  0000 C CNN
+F 1 "BY399" H 5750 2900 50  0000 C CNN
 F 2 "" H 5550 2950 60  0001 C CNN
 F 3 "" H 5550 2950 60  0001 C CNN
@@
 U 1 1 4DD3E61D
 P 4750 3600
-F 0 "D12" H 4850 3700 40  0000 C CNN
-F 1 "BY399" V 4400 3600 40  0000 C CNN
+F 0 "D12" V 4850 3700 50  0000 C CNN
+F 1 "BY399" V 4400 3600 50  0000 C CNN
 F 2 "" H 4750 3600 60  0001 C CNN
 F 3 "" H 4750 3600 60  0001 C CNN
@@
 U 1 1 4DD3E3EE
 P 4750 2400
-F 0 "D6" H 4650 2500 40  0000 C CNN
-F 1 "1N4001" V 5100 2400 40  0000 C CNN
+F 0 "D6" V 4650 2500 50  0000 C CNN
+F 1 "1N4001" V 5100 2400 50  0000 C CNN
 F 2 "" H 4750 2400 60  0001 C CNN
 F 3 "" H 4750 2400 60  0001 C CNN
@@
 U 1 1 4DD3E3E9
 P 5550 1750
-F 0 "D5" H 5650 1850 40  0000 C CNN
+F 0 "D5" H 5650 1850 50  0000 C CNN
 F 1 "1N4001" H 5350 1700 50  0000 C CNN
 F 2 "" H 5550 1750 60  0001 C CNN
@@
 U 1 1 4DD3E28F
 P 6950 2300
-F 0 "D3" H 6800 2250 40  0000 C CNN
+F 0 "D3" H 6800 2250 50  0000 C CNN
 F 1 "1N4001" H 6950 2000 40  0001 C CNN
 F 2 "" H 6950 2300 60  0001 C CNN
@@
 U 1 1 4DD3E290
 P 6950 2150
-F 0 "D1" H 7100 2200 40  0000 C CNN
-F 1 "1N4001" H 6950 1550 40  0000 C CNN
+F 0 "D1" H 7100 2200 50  0000 C CNN
+F 1 "1N4001" H 6950 1550 50  0000 C CNN
 F 2 "" H 6950 2150 60  0001 C CNN
 F 3 "" H 6950 2150 60  0001 C CNN
@@
 U 1 1 4DD3E28E
 P 6950 2600
-F 0 "D4" H 6800 2550 40  0000 C CNN
+F 0 "D4" H 6800 2550 50  0000 C CNN
 F 1 "1N4001" H 7150 2400 40  0001 C CNN
 F 2 "" H 6950 2600 60  0001 C CNN
@@
 U 1 1 4DD3E28D
 P 6950 2450
-F 0 "D2" H 7100 2500 40  0000 C CNN
+F 0 "D2" H 7100 2500 50  0000 C CNN
 F 1 "1N4001" H 6750 2350 40  0001 C CNN
 F 2 "" H 6950 2450 60  0001 C CNN

Commit message: 220911
Connections:
- net labels added: -NPN/PNP
- net labels removed: -NPN
Changed lines of the file:
@@
 Text Notes 3350 5100 0    60   ~ 0
 CN3
-Text Notes 8100 6190 0    60   ~ 0
+Text Notes 7900 6350 0    60   ~ 0
 CN4
 Text Notes 3350 3000 0    60   ~ 0
@@
 POL
 Text HLabel 7650 6150 2    60   Input ~ 0
--NPN
+-NPN/PNP
 Text HLabel 3850 4800 0    60   Output ~ 0
 +Um2
