File: cad_files/ctt_ps/ctt_ps3.sch (KiCad schematic (older format))
At the start: 55 parts, among them IC1 DAC0832, IC10 OPTONPN, IC11 74LS374, IC2 LF351, IC3 OPTONPN, IC4 OPTONPN, IC5 OPTONPN, IC6 OPTONPN, IC7 OPTONPN, IC8 OPTONPN, IC9 OPTONPN, J1 RELAY, P1 100k, T1 BC212, T2 BC212, T3 BC212, T4 BC109, T5 BC182

Commit message: 220902
Parts:
- C1, C2, C3, C6: symbol CP -> CP-RESCUE-ctt
- C4, C5: symbol C -> C-RESCUE-ctt
- IC2: symbol LM741 -> LM741-RESCUE-ctt
- P1: symbol POT -> POT-RESCUE-ctt
- R1, R10, R11, R12, R13, R14, R15, R16, R17, R18, R19, R2, R20, R21, R22, R23, R24, R3, R4, R5, R6, R7, R8, R9: symbol R -> R-RESCUE-ctt
Connections:
- wire segments 286 -> 207

Commit message: 220911
Parts:
- removed C4: 33n, symbol C-RESCUE-ctt
- removed C6: 10u, symbol CP-RESCUE-ctt
- removed D5: 1,2V, symbol ZENER
- removed IC1: DAC0832, symbol DAC0832
- removed IC10, IC3, IC4, IC5, IC6, IC7, IC8, IC9: OPTONPN, symbol OPTONPN
- removed IC11: 74LS374, symbol 74LS374
- removed IC2: LF351, symbol LM741-RESCUE-ctt
- removed J1: RELAY, symbol RELAY
- removed JC1, JC2: SWITCH_INV, symbol SWITCH_INV
- removed P1: 100k, symbol POT-RESCUE-ctt
- removed R1: 300, symbol R-RESCUE-ctt
- removed R10, R11, R12, R13, R14, R15, R8, R9: 4,7k, symbol R-RESCUE-ctt
- removed R16, R17, R18, R19, R20, R21, R22, R23, R6, R7: 1k, symbol R-RESCUE-ctt
- removed R2: 12, symbol R-RESCUE-ctt
- removed R24: 470, symbol R-RESCUE-ctt
- removed R3, R4: 1,5K, symbol R-RESCUE-ctt
- removed R5: 4,3k, symbol R-RESCUE-ctt
- removed T1, T2, T3: BC212, symbol PNP
- added C4: 100u, symbol CP-RESCUE-ctt
- added D10, D11, D12, D13, D14, D15, D16, D5, D7, D8, D9: 1N4001, symbol DIODE
- added D6: ZPD3,3, symbol ZENER
- added IC1: LM317L, TO-92, symbol LM317T
- added IC2: 74LS374, symbol 74LS374
- added K1: LMR2-5D, symbol Relay_LMR2-5D
- added K2, K3, K4, K5, K6, K7, K8, K9: LEG-5, symbol Relay_LEG-5
- added P1: 390, symbol POT
- added R1: 640, symbol R
- added R10, R11, R12, R13, R14, R15, R16, R17, R18: 1k, symbol R
- added R2: 2, symbol R
- added R3: 4, symbol R
- added R4: 8, symbol R
- added R5: 16, symbol R
- added R6: 32, symbol R
- added R7: 64, symbol R
- added R8: 128, symbol R
- added R9: 256, symbol R
- added T1, T2, T3, T6, T7, T8, T9: BC109, symbol NPN
- C1: value 2200u 16V -> 2200u; Voltage (none) -> 40V
- C2: value 2200u 16V -> 1u; Voltage (none) -> 40V
- C3: value 10u 6V -> 470u; Voltage (none) -> 40V
- C5: value 33n -> 100n
- D1, D2, D3, D4: value BY399 -> 1N4001
- T5: value BC182 -> BC109
Connections:
- net labels added: GND-RESCUE-ctt, Um1
- net labels removed: Um3
- wire segments 207 -> 199
- no-connect marks 0 -> 8
Other:
- note added: "CN1"
- note added: "CN2"
- note added: "CN3"
- note added: "CN4"
- note added: "CN5"
- note added: "CN6"
- note removed: ""set zero""
- note removed: "ISOLATED PART"

Commit message: 220912
Parts:
- added C5: 100u, symbol CP-RESCUE-ctt
- C1: value 2200u -> 470u; Voltage 40V -> 16V
- C2: value 1u -> 10u; Voltage 40V -> 16V
- C3: value 470u -> 10u; Voltage 40V -> 16V
- C4: value 100u -> 470u; Voltage 10V -> 16V
- D1, D4: value 1N4001 -> 1N4002
- renumbered C5 to C6
Connections:
- net 5V 100mA AC COM: now also C3.2, C4.1; no longer C3.1, D4.1 (A)
- net GND: now also C5.2; no longer C4.2
- net VCC: now also C6.1, D10.2 (K), D11.2 (K), D12.2 (K), D13.2 (K), D14.2 (K), D15.2 (K), D16.2 (K), D5.2 (K), D9.2 (K), K1.1 (Coil), K2.1 (Coil), K3.1 (Coil), K4.1 (Coil), K5.1 (Coil), K6.1 (Coil), K7.1 (Coil), K8.1 (Coil), K9.1 (Coil), C5.1
- net at IC1.1 (ADJ), K9.3 (Common), R1.2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: now also C3.1, D4.1 (A)
- net at D6.1 (A), D7.1 (A), D8.1 (A): now also C4.2; no longer C3.2
- removed net +5V: C4.1, C6.1, D10.2 (K), D11.2 (K), D12.2 (K), D13.2 (K), D14.2 (K), D15.2 (K), D16.2 (K), D5.2 (K), D9.2 (K), K1.1 (Coil), K2.1 (Coil), K3.1 (Coil), K4.1 (Coil), K5.1 (Coil), K6.1 (Coil), K7.1 (Coil), K8.1 (Coil), K9.1 (Coil)
