File: cad_files/ctt_ps/ctt_ps2.sch (KiCad schematic (older format))
At the start: 55 parts, among them IC1 DAC0832, IC10 OPTONPN, IC11 74LS374, IC2 LF351, IC3 OPTONPN, IC4 OPTONPN, IC5 OPTONPN, IC6 OPTONPN, IC7 OPTONPN, IC8 OPTONPN, IC9 OPTONPN, J1 RELAY, P1 100k, T1 BC212, T2 BC212, T3 BC212, T4 BC109, T5 BC182

Commit message: 220902
Parts:
- C1, C2, C3, C6: symbol CP -> CP-RESCUE-ctt
- C4, C5: symbol C -> C-RESCUE-ctt
- IC2: symbol LM741 -> LM741-RESCUE-ctt
- P1: symbol POT -> POT-RESCUE-ctt
- R1, R10, R11, R12, R13, R14, R15, R16, R17, R18, R19, R2, R20, R21, R22, R23, R24, R3, R4, R5, R6, R7, R8, R9: symbol R -> R-RESCUE-ctt
Connections:
- wire segments 285 -> 208

Commit message: 220910
Parts:
- removed C4: 33n, symbol C-RESCUE-ctt
- removed C6: 10u, symbol CP-RESCUE-ctt
- removed IC1: DAC0832, symbol DAC0832
- removed IC10, IC3, IC4, IC5, IC6, IC7, IC8, IC9: OPTONPN, symbol OPTONPN
- removed IC11: 74LS374, symbol 74LS374
- removed IC2: LF351, symbol LM741-RESCUE-ctt
- removed J1: RELAY, symbol RELAY
- removed P1: 100k, symbol POT-RESCUE-ctt
- removed R1: 300, symbol R-RESCUE-ctt
- removed R10, R11, R12, R13, R14, R15, R8, R9: 4,7k, symbol R-RESCUE-ctt
- removed R16, R17, R18, R19, R20, R21, R22, R23, R6, R7: 1k, symbol R-RESCUE-ctt
- removed R2: 12, symbol R-RESCUE-ctt
- removed R24: 470, symbol R-RESCUE-ctt
- removed R3, R4: 1,5K, symbol R-RESCUE-ctt
- removed R5: 4,3k, symbol R-RESCUE-ctt
- removed T1, T2, T3: BC212, symbol PNP
- added C4: 100u, symbol CP-RESCUE-ctt
- added D10, D11, D12, D13, D14, D15, D16, D8, D9: 1N4001, symbol DIODE
- added D6, D7: BY399, symbol DIODE
- added IC1: 74LS374, symbol 74LS374
- added IC2: LM317T, TO-220, symbol LM317T
- added K1, K2, K3, K4, K5, K6, K7, K8, K9: RELAY, symbol RELAY
- added K1a, K2a, K3a, K4a, K5a, K6a, K7a, K8a: SPST, symbol SPST
- added P1: POT, symbol POT
- added R1, R10, R2, R3, R4, R5, R6, R7, R8, R9: R, symbol R
- added R11, R12, R13, R14, R15, R16, R17, R18, R19: 1k, symbol R
- added T1, T2, T3, T6, T7, T8, T9: BC109, symbol NPN
- C1: value 2200u 16V -> 2200u; Voltage (none) -> 40V
- C2: value 2200u 16V -> 1u
- C3: value 10u 6V -> 470u; Voltage (none) -> 40V
- C5: value 33n -> 100n
- D4: value BY399 -> 1N4001
- D5: value 1,2V -> ZENER
- T5: value BC182 -> BC109
- renumbered JC1 to K9a1, JC2 to K9b1
Connections:
- net labels added: GND-RESCUE-ctt
- wire segments 208 -> 261
Other:
- note added: "CN1"
- note added: "CN2"
- note added: "CN3"
- note added: "CN4"
- note added: "CN5"
- note added: "CN6"
- note added: "CN7"
- note removed: ""set zero""
- note removed: "ISOLATED PART"
- moved on the sheet: C1, C2, D3

Commit message: 220911
Parts:
- removed K1a, K2a, K3a, K4a, K5a, K6a, K7a, K8a: SPST, symbol SPST
- removed K2, K3, K4, K5, K6, K7, K8, K9: RELAY, symbol RELAY
- added K2, K3, K4, K5, K6, K7, K8, K9: LEG-5, symbol Relay_LEG-5
- C2: Voltage (none) -> 40V
- D5: value ZENER -> ZPD3.3
- R1, R7: value R -> 320
- R10: value R -> 2560
- R3: value R -> 20
- R4: value R -> 40
- R5: value R -> 80
- R6: value R -> 160
- R8: value R -> 640
- R9: value R -> 1280
Connections:
- wire segments 261 -> 276
- no-connect marks 0 -> 8
Other:
- note removed: "CN7"
- moved on the sheet: C1, C2, C3, C4, C5, D1, D2, D3, D4, D5, D6, D7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

Commit message: 220911
Parts:
- removed K1: RELAY, symbol RELAY
- removed K9a1, K9b1: SWITCH_INV, symbol SWITCH_INV
- removed R2: R, symbol R
- added K1: LMR2-5D, symbol Relay_LMR2-5D
- D6: renamed from D5; value ZPD3.3 -> ZPD27
- P1: value POT -> 390
- renumbered D9 to D5, D6 to D7, D7 to D8, D8 to D9, IC2 to IC1, IC1 to IC2, R11 to R10, R12 to R11, R13 to R12, R14 to R13, R15 to R14, R16 to R15, R17 to R16, R18 to R17, R19 to R18, R3 to R2, R4 to R3, R5 to R4, R6 to R5, R7 to R6, R8 to R7, R9 to R8, R10 to R9
Connections:
- wire segments 276 -> 275
Other:
- moved on the sheet: D5, D6, P1

Commit message: 220912
Parts:
- removed C5: 100n, symbol C-RESCUE-ctt
- added C3: 10u, symbol CP-RESCUE-ctt
- added C6: 100n, symbol C-RESCUE-ctt
- C2: value 1u -> 10u
- D1: value BY399 -> 1N4002
- D4: value 1N4001 -> 1N4002
- renumbered C3 to C4, C4 to C5
Connections:
- net +5V is gone; now on net VCC: C5.1, D10.2 (K), D11.2 (K), D12.2 (K), D13.2 (K), D14.2 (K), D15.2 (K), D16.2 (K), D5.2 (K), D9.2 (K), K1.1 (Coil), K2.1 (Coil), K3.1 (Coil), K4.1 (Coil), K5.1 (Coil), K6.1 (Coil), K7.1 (Coil), K8.1 (Coil), K9.1 (Coil)
- net 25V 1A AC COM: now also C3.2; no longer D4.1 (A)
- net GND: now also C6.2
- net VCC: now also C6.1
- net at IC1.1 (ADJ), K9.3 (Common), R1.2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: now also D4.1 (A), C3.1
Other:
- moved on the sheet: D4

Commit message: 220914
Parts:
- C6: footprint (none) -> Capacitors_THT:C_Disc_D6.0mm_W2.5mm_P5.00mm
- D1, D10, D11, D12, D13, D14, D15, D16, D4, D5, D6, D7, D8, D9: footprint (none) -> Diodes_THT:D_A-405_P12.70mm_Horizontal
- D2, D3: footprint (none) -> Diodes_THT:D_5W_P12.70mm_Horizontal
- IC1: footprint TO-220 -> Power_Integrations:TO-220
- IC2: footprint (none) -> Housings_DIP:DIP-20_W7.62mm_LongPads
- K2, K3, K4, K5, K6, K7, K8, K9: footprint (none) -> relay_lg:relay_leg
- R10, R11, R12, R13, R14, R15, R16, R17, R18: footprint (none) -> Resistors_THT:R_Axial_DIN0207_L6.3mm_D2.5mm_P10.16mm_Horizontal
- T1, T2, T3, T4, T5, T6, T7, T8, T9: footprint (none) -> TO_SOT_Packages_THT:TO-18-3
