File: cad_files/ctt_ps2/ctt_ps2.kicad_pcb (KiCad board)
At the start: 2 copper layers, 141 x 73.7 mm, 61 parts, among them IC1 LM317T, IC2 74LS374, K1 LMR2-5D, K2 LEG-5, K3 LEG-5, K4 LEG-5, K5 LEG-5, K6 LEG-5, K7 LEG-5, K8 LEG-5, K9 LEG-5, P1 390, T1 BC109, T2 BC109, T3 BC109, T4 BC109, T5 BC109, T6 BC109, T7 BC109, T8 BC109, T9 BC109

Commit message: 220919
Parts:
- D5: footprint Diodes_THT:D_A-405_P12.70mm_Horizontal -> Diodes_THT:D_A-405_P10.16mm_Horizontal
- D7, D8: value BY399 -> 1N4001
- R1, R2, R3, R4, R5, R6, R7, R8, R9: footprint Resistors_THT:R_Axial_DIN0414_L11.9mm_D4.5mm_P15.24mm_Horizontal -> Resistors_THT:R_Axial_DIN0411_L9.9mm_D3.6mm_P12.70mm_Horizontal
- R10, R11, R12, R13, R14, R15, R16, R17, R18: footprint Resistors_THT:R_Axial_DIN0207_L6.3mm_D2.5mm_P10.16mm_Horizontal -> Resistors_THT:R_Axial_DIN0411_L9.9mm_D3.6mm_P5.08mm_Vertical
- moved K1 302.9 mm to (94.0, 124.5), turned to 0 degrees
- moved R9 268.6 mm to (141.0, 128.3), turned to 0 degrees
- moved R18 264.7 mm to (128.3, 127.0)
- moved T9 258.6 mm to (134.6, 128.3)
- moved R8 243.1 mm to (158.8, 128.3), turned to 0 degrees
- moved K9 238.3 mm to (147.3, 113.7), turned to 270 degrees
- moved R17 232.9 mm to (128.3, 96.5)
- moved D16 230.8 mm to (141.0, 99.1), turned to 0 degrees
- moved T8 226.1 mm to (134.6, 97.8)
- moved R7 220.9 mm to (176.5, 128.3), turned to 0 degrees
- moved R16 220.2 mm to (128.3, 104.1)
- moved T7 213.2 mm to (134.6, 105.4)
- moved K8 211.6 mm to (165.1, 113.7), turned to 270 degrees
- moved R15 208.8 mm to (128.3, 111.8)
- moved D5 206.5 mm to (111.8, 129.5), turned to 90 degrees
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Connections:
- K1 pad 3: (no net) -> /25V 1A AC COM
- K1 pad 6: (no net) -> /25V 1A AC COM
- K1 pad 7: (no net) -> /Um3
- K1 pad 8: (no net) -> Net-(C2-Pad1)
- T1 pad 1: Net-(T1-Pad1) -> GND
- T2 pad 1: Net-(T1-Pad1) -> GND
- T3 pad 1: Net-(T1-Pad1) -> GND
- T4 pad 1: Net-(T1-Pad1) -> GND
- T5 pad 1: Net-(T1-Pad1) -> GND
- T6 pad 1: Net-(T1-Pad1) -> GND
- T7 pad 1: Net-(T1-Pad1) -> GND
- T8 pad 1: Net-(T1-Pad1) -> GND
- T9 pad 1: Net-(T1-Pad1) -> GND
Routing:
- net VCC: track 0.00 -> 171.9 mm
- net GND: track 0.00 -> 119.3 mm
- net Net-(D12-Pad1): track 0.00 -> 97.9 mm
- net Net-(K5-Pad3): track 0.00 -> 96.6 mm
- net Net-(D13-Pad1): track 0.00 -> 77.6 mm
- net Net-(IC2-Pad9): track 0.00 -> 76.5 mm
- net Net-(D11-Pad1): track 0.00 -> 73.2 mm
- net Net-(D14-Pad1): track 0.00 -> 61.6 mm
- net Net-(IC2-Pad6): track 0.00 -> 61.3 mm
- net Net-(IC2-Pad5): track 0.00 -> 51.1 mm
- net Net-(D10-Pad1): track 0.00 -> 49.3 mm
- net Net-(D15-Pad1): track 0.00 -> 48.1 mm
- net Net-(IC2-Pad12): track 0.00 -> 44.2 mm
- net Net-(K8-Pad3): track 0.00 -> 40.8 mm
- net Net-(K7-Pad3): track 0.00 -> 40.8 mm
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
Commit message: 220920
Parts:
- added CN3: Pin_Header_Straight_1x08, Pin_Headers:Pin_Header_Straight_1x08, F.Cu at (104.1, 96.5)
- added CN4: Pin_Header_Straight_1x01, Pin_Headers:Pin_Header_Straight_1x01, F.Cu at (81.3, 96.5)
- added CN5: Pin_Header_Straight_1x01, Pin_Headers:Pin_Header_Straight_1x01, F.Cu at (109.2, 96.5)
- added REF**: Pin_Header_Straight_1x01, Pin_Headers:Pin_Header_Straight_1x01, F.Cu at (118.1, 129.5)
- added REF**: Pin_Header_Straight_1x02, Pin_Headers:Pin_Header_Straight_1x02, F.Cu at (88.9, 92.7)
- added REF**: Pin_Header_Straight_1x03, Pin_Headers:Pin_Header_Straight_1x03, F.Cu at (85.1, 66.0)
- moved C5 182.4 mm to (116.2, 111.8), turned to 90 degrees
- moved C2 172.3 mm to (114.3, 86.4), turned to 180 degrees
- moved P1 160.6 mm to (104.1, 66.0), turned to 270 degrees
- moved C3 156.7 mm to (114.3, 92.7), turned to 180 degrees
- moved D4 155.8 mm to (114.3, 69.8), turned to 270 degrees
- moved D8 141.4 mm to (92.7, 71.1), turned to 270 degrees
- moved IC1 133.9 mm to (114.3, 66.0)
- moved D6 132.1 mm to (80.0, 88.9)
- moved D7 127.6 mm to (80.0, 71.1), turned to 270 degrees
- moved D1 125.4 mm to (116.8, 69.8)
- moved D3 123.6 mm to (88.9, 83.8), turned to 90 degrees
- moved C4 122.0 mm to (104.1, 73.7), turned to 180 degrees
- moved D2 116.2 mm to (83.8, 83.8), turned to 90 degrees
- moved C1 109.3 mm to (97.8, 86.4)
- moved R1 105.5 mm to (110.5, 82.5), turned to 90 degrees
Connections:
- D1 pad 1: Net-(C2-Pad1) -> Net-(C1-Pad1)
- D1 pad 2: Net-(C1-Pad1) -> Net-(C2-Pad1)
- D10 pad 1: Net-(D10-Pad1) -> VCC
- D10 pad 2: VCC -> Net-(D10-Pad2)
- D11 pad 1: Net-(D11-Pad1) -> VCC
- D11 pad 2: VCC -> Net-(D11-Pad2)
- D12 pad 1: Net-(D12-Pad1) -> VCC
- D12 pad 2: VCC -> Net-(D12-Pad2)
- D13 pad 1: Net-(D13-Pad1) -> VCC
- D13 pad 2: VCC -> Net-(D13-Pad2)
- D14 pad 1: Net-(D14-Pad1) -> VCC
- D14 pad 2: VCC -> Net-(D14-Pad2)
- D15 pad 1: Net-(D15-Pad1) -> VCC
- D15 pad 2: VCC -> Net-(D15-Pad2)
- D16 pad 1: Net-(D16-Pad1) -> VCC
- D16 pad 2: VCC -> Net-(D16-Pad2)
- D2 pad 1: /25V 1A AC -> Net-(C1-Pad1)
- D2 pad 2: Net-(C1-Pad1) -> /25V 1A AC
- D3 pad 1: /25V 1A AC -> Net-(C1-Pad1)
- D3 pad 2: Net-(C1-Pad1) -> /25V 1A AC
- D4 pad 1: Net-(C3-Pad1) -> Net-(C2-Pad1)
- D4 pad 2: Net-(C2-Pad1) -> Net-(C3-Pad1)
- D5 pad 1: Net-(D5-Pad1) -> VCC
- D5 pad 2: VCC -> Net-(D5-Pad2)
- D7 pad 1: Net-(C4-Pad2) -> /25V 1A AC
- D7 pad 2: /25V 1A AC -> Net-(C4-Pad2)
- D8 pad 1: Net-(C4-Pad2) -> /25V 1A AC
- D8 pad 2: /25V 1A AC -> Net-(C4-Pad2)
- D9 pad 1: Net-(D9-Pad1) -> VCC
- D9 pad 2: VCC -> Net-(D9-Pad2)
- K1 pad 2: Net-(D5-Pad1) -> Net-(D5-Pad2)
- K2 pad 2: Net-(D9-Pad1) -> Net-(D9-Pad2)
- K3 pad 2: Net-(D10-Pad1) -> Net-(D10-Pad2)
- K4 pad 2: Net-(D11-Pad1) -> Net-(D11-Pad2)
- K5 pad 2: Net-(D12-Pad1) -> Net-(D12-Pad2)
- K6 pad 2: Net-(D13-Pad1) -> Net-(D13-Pad2)
- K7 pad 2: Net-(D14-Pad1) -> Net-(D14-Pad2)
- K8 pad 2: Net-(D15-Pad1) -> Net-(D15-Pad2)
- K9 pad 2: Net-(D16-Pad1) -> Net-(D16-Pad2)
- T1 pad 3: Net-(D9-Pad1) -> Net-(D9-Pad2)
- T2 pad 3: Net-(D10-Pad1) -> Net-(D10-Pad2)
- T3 pad 3: Net-(D11-Pad1) -> Net-(D11-Pad2)
- T4 pad 3: Net-(D12-Pad1) -> Net-(D12-Pad2)
- T5 pad 3: Net-(D13-Pad1) -> Net-(D13-Pad2)
- T6 pad 3: Net-(D14-Pad1) -> Net-(D14-Pad2)
- T7 pad 3: Net-(D15-Pad1) -> Net-(D15-Pad2)
- T8 pad 3: Net-(D16-Pad1) -> Net-(D16-Pad2)
- T9 pad 3: Net-(D5-Pad1) -> Net-(D5-Pad2)
Routing:
- net Net-(D12-Pad2): track 0.00 -> 108.0 mm
- net Net-(D9-Pad2): track 0.00 -> 107.8 mm
- net Net-(D12-Pad1): track 97.9 -> 0.00 mm
- net Net-(D11-Pad2): track 0.00 -> 83.4 mm
- net Net-(D13-Pad1): track 77.6 -> 0.00 mm
- net Net-(D11-Pad1): track 73.2 -> 0.00 mm
- net Net-(D13-Pad2): track 0.00 -> 69.5 mm
- net VCC: track 171.9 -> 107.9 mm
- net Net-(D14-Pad1): track 61.6 -> 0.00 mm
- net /25V 1A AC COM: track 16.3 -> 75.1 mm
- net Net-(D10-Pad2): track 0.00 -> 56.9 mm
- net Net-(C3-Pad1): track 27.8 -> 84.3 mm
- net Net-(D14-Pad2): track 0.00 -> 54.8 mm
- net Net-(D10-Pad1): track 49.3 -> 0.00 mm
- net Net-(D15-Pad1): track 48.1 -> 0.00 mm
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
Commit message: 220920
Parts:
- moved CN2 39.6 mm to (118.1, 119.4), turned to 0 degrees
- moved P1 5.08 mm to (99.1, 66.0), turned to 90 degrees
- moved C2 0.64 mm to (114.3, 87.0)
- renumbered REF** to CN1, REF** to CN2, REF** to CN6
Routing:
- net Net-(C2-Pad1): track 31.1 -> 118.5 mm
- net GND: track 132.8 -> 196.0 mm
- net Net-(C3-Pad1): track 84.3 -> 133.2 mm, vias 0 -> 1
- net /25V 1A AC COM: track 75.1 -> 115.5 mm
- net Net-(C1-Pad1): track 18.8 -> 52.9 mm
- net Net-(D6-Pad2): track 27.0 -> 57.2 mm
- net Net-(C4-Pad2): track 36.6 -> 23.9 mm
- net VCC: track 107.9 -> 116.7 mm
Other:
- board text added: "CTT/PS2-3"
- board text added: "DN: CTT/25-27"
- board text added: "http://www.pozsarzs.hu"
