File: cad_files/ctt_ps2/ctt_ps2.sch (KiCad schematic (older format))
At the start: 61 parts, among them IC1 LM317T, IC2 74LS374, K1 LMR2-5D, K2 LEG-5, K3 LEG-5, K4 LEG-5, K5 LEG-5, K6 LEG-5, K7 LEG-5, K8 LEG-5, K9 LEG-5, P1 390, T1 BC109, T2 BC109, T3 BC109, T4 BC109, T5 BC109, T6 BC109, T7 BC109, T8 BC109, T9 BC109

Commit message: 220915
Other:
- note added: "1"
- note added: "2"
- note added: "3"
- note added: "4"
- note added: "5"
- note added: "6"
- note added: "7"
- note added: "8"
Changed lines of the file:
@@
 EESchema Schematic File Version 2
+LIBS:ctt-rescue
 LIBS:power
 LIBS:device
-LIBS:transistors
 LIBS:conn
 LIBS:linear
@@
 LIBS:cypress
 LIBS:siliconi
-LIBS:opto
-LIBS:atmel
 LIBS:contrib
 LIBS:valves
 LIBS:ctt-cache
-LIBS:ctt-rescue
-LIBS:relay_leg-5
 EELAYER 25 0
 EELAYER END
 $Descr A4 11693 8268
 encoding utf-8
-Sheet 1 1
+Sheet 4 11
 Title "CTT Transistor tester - CTT/PS2 power supply unit"
 Date "28 jan 2012"
@@
 	-1   0    0    -1
 $EndComp
+Text Notes 1650 4875 0    60   ~ 0
+1
+Text Notes 1650 4975 0    60   ~ 0
+2
+Text Notes 1650 5075 0    60   ~ 0
+3
+Text Notes 1650 5175 0    60   ~ 0
+4
+Text Notes 1650 5275 0    60   ~ 0
+5
+Text Notes 1650 5375 0    60   ~ 0
+6
+Text Notes 1650 5475 0    60   ~ 0
+7
+Text Notes 1650 5575 0    60   ~ 0
+8
+Text Notes 1650 1650 0    60   ~ 0
+1
+Text Notes 1650 2550 0    60   ~ 0
+3
+Text Notes 1650 3450 0    60   ~ 0
+2
+Text Notes 1650 3750 0    60   ~ 0
+1
+Text Notes 1650 4350 0    60   ~ 0
+2
+Text Notes 1650 5775 0    60   ~ 0
+1
+Text Notes 1650 6125 0    60   ~ 0
+1
+Text Notes 10050 1900 0    60   ~ 0
+1
 $EndSCHEMATC

Commit message: 220918
Parts:
- C1: footprint (none) -> Capacitors_THT:CP_Radial_D14.0mm_P7.50mm
- C2, C3: footprint (none) -> Capacitors_THT:CP_Radial_D5.0mm_P2.50mm
- C4, C5: footprint (none) -> Capacitors_THT:CP_Radial_D10.0mm_P5.00mm
- K1: footprint (none) -> relay_lmr2:relay_lmr2
- K2, K3, K4, K5, K6, K7, K8, K9: footprint relay_lg:relay_leg -> relay_leg:relay_leg
- P1: footprint (none) -> Potentiometers:Potentiometer_WirePads_Small
- R1, R2, R3, R4, R5, R6, R7, R8, R9: footprint (none) -> Resistors_THT:R_Axial_DIN0414_L11.9mm_D4.5mm_P15.24mm_Horizontal

Commit message: 220919
Parts:
- D5: footprint Diodes_THT:D_A-405_P12.70mm_Horizontal -> Diodes_THT:D_A-405_P10.16mm_Horizontal
- D7, D8: value BY399 -> 1N4001
- R1, R2, R3, R4, R5, R6, R7, R8, R9: footprint Resistors_THT:R_Axial_DIN0414_L11.9mm_D4.5mm_P15.24mm_Horizontal -> Resistors_THT:R_Axial_DIN0411_L9.9mm_D3.6mm_P12.70mm_Horizontal
- R10, R11, R12, R13, R14, R15, R16, R17, R18: footprint Resistors_THT:R_Axial_DIN0207_L6.3mm_D2.5mm_P10.16mm_Horizontal -> Resistors_THT:R_Axial_DIN0411_L9.9mm_D3.6mm_P5.08mm_Vertical
Connections:
- net GND: now also T1.1 (E), T2.1 (E), T3.1 (E), T4.1 (E), T5.1 (E), T6.1 (E), T7.1 (E), T8.1 (E), T9.1 (E)
Changed lines of the file:
@@
 EESchema Schematic File Version 2
+LIBS:ctt-rescue
 LIBS:power
 LIBS:device
-LIBS:transistors
 LIBS:conn
 LIBS:linear
@@
 LIBS:cypress
 LIBS:siliconi
-LIBS:opto
-LIBS:atmel
 LIBS:contrib
 LIBS:valves
 LIBS:ctt-cache
-LIBS:ctt-rescue
-LIBS:relay_leg-5
-LIBS:ctt_ps2-cache
 EELAYER 25 0
 EELAYER END
 $Descr A4 11693 8268
 encoding utf-8
-Sheet 1 1
+Sheet 4 11
 Title "CTT Transistor tester - CTT/PS2 power supply unit"
 Date "28 jan 2012"
 Rev "1.0"
 Comp "Pozsar Zsolt"
-Comment1 "Draw number: CTT/34"
+Comment1 "Draw number: CTT/24"
 Comment2 ""
 Comment3 ""
@@
 F 0 "R2" V 5150 3150 50  0000 C CNN
 F 1 "20" V 5150 3300 50  0000 C CNN
-F 2 "Resistors_THT:R_Axial_DIN0414_L11.9mm_D4.5mm_P15.24mm_Horizontal" V 5180 3250 50  0001 C CNN
+F 2 "Resistors_THT:R_Axial_DIN0411_L9.9mm_D3.6mm_P12.70mm_Horizontal" V 5180 3250 50  0001 C CNN
 F 3 "" H 5250 3250 50  0000 C CNN
 	1    5250 3250
@@
 F 0 "R1" V 3900 1950 50  0000 C CNN
 F 1 "320" V 3900 2100 50  0000 C CNN
-F 2 "Resistors_THT:R_Axial_DIN0414_L11.9mm_D4.5mm_P15.24mm_Horizontal" V 3930 2050 50  0001 C CNN
+F 2 "Resistors_THT:R_Axial_DIN0411_L9.9mm_D3.6mm_P12.70mm_Horizontal" V 3930 2050 50  0001 C CNN
 F 3 "" H 4000 2050 50  0000 C CNN
 	1    4000 2050
@@
 F 0 "R10" V 4750 4675 50  0000 C CNN
 F 1 "1k" V 4750 5075 50  0000 C CNN
-F 2 "Resistors_THT:R_Axial_DIN0207_L6.3mm_D2.5mm_P10.16mm_Horizontal" V 4730 4875 50  0001 C CNN
+F 2 "Resistors_THT:R_Axial_DIN0411_L9.9mm_D3.6mm_P5.08mm_Vertical" V 4730 4875 50  0001 C CNN
 F 3 "" H 4800 4875 50  0000 C CNN
 	1    4800 4875
@@
 F 0 "R11" V 4750 4775 50  0000 C CNN
 F 1 "1k" V 4750 5175 50  0000 C CNN
-F 2 "Resistors_THT:R_Axial_DIN0207_L6.3mm_D2.5mm_P10.16mm_Horizontal" V 4730 4975 50  0001 C CNN
+F 2 "Resistors_THT:R_Axial_DIN0411_L9.9mm_D3.6mm_P5.08mm_Vertical" V 4730 4975 50  0001 C CNN
 F 3 "" H 4800 4975 50  0000 C CNN
 	1    4800 4975
@@
 F 0 "R12" V 4750 4875 50  0000 C CNN
 F 1 "1k" V 4750 5275 50  0000 C CNN
-F 2 "Resistors_THT:R_Axial_DIN0207_L6.3mm_D2.5mm_P10.16mm_Horizontal" V 4730 5075 50  0001 C CNN
+F 2 "Resistors_THT:R_Axial_DIN0411_L9.9mm_D3.6mm_P5.08mm_Vertical" V 4730 5075 50  0001 C CNN
 F 3 "" H 4800 5075 50  0000 C CNN
 	1    4800 5075
@@
 F 0 "R13" V 4750 4975 50  0000 C CNN
 F 1 "1k" V 4750 5375 50  0000 C CNN
-F 2 "Resistors_THT:R_Axial_DIN0207_L6.3mm_D2.5mm_P10.16mm_Horizontal" V 4730 5175 50  0001 C CNN
+F 2 "Resistors_THT:R_Axial_DIN0411_L9.9mm_D3.6mm_P5.08mm_Vertical" V 4730 5175 50  0001 C CNN
 F 3 "" H 4800 5175 50  0000 C CNN
 	1    4800 5175
@@
 F 0 "R14" V 4750 5075 50  0000 C CNN
 F 1 "1k" V 4750 5475 50  0000 C CNN
-F 2 "Resistors_THT:R_Axial_DIN0207_L6.3mm_D2.5mm_P10.16mm_Horizontal" V 4730 5275 50  0001 C CNN
+F 2 "Resistors_THT:R_Axial_DIN0411_L9.9mm_D3.6mm_P5.08mm_Vertical" V 4730 5275 50  0001 C CNN
 F 3 "" H 4800 5275 50  0000 C CNN
 	1    4800 5275
@@
 F 0 "R15" V 4750 5175 50  0000 C CNN
 F 1 "1k" V 4750 5575 50  0000 C CNN
-F 2 "Resistors_THT:R_Axial_DIN0207_L6.3mm_D2.5mm_P10.16mm_Horizontal" V 4730 5375 50  0001 C CNN
+F 2 "Resistors_THT:R_Axial_DIN0411_L9.9mm_D3.6mm_P5.08mm_Vertical" V 4730 5375 50  0001 C CNN
 F 3 "" H 4800 5375 50  0000 C CNN
 	1    4800 5375
@@
 F 0 "R16" V 4750 5275 50  0000 C CNN
 F 1 "1k" V 4750 5675 50  0000 C CNN
-F 2 "Resistors_THT:R_Axial_DIN0207_L6.3mm_D2.5mm_P10.16mm_Horizontal" V 4730 5475 50  0001 C CNN
+F 2 "Resistors_THT:R_Axial_DIN0411_L9.9mm_D3.6mm_P5.08mm_Vertical" V 4730 5475 50  0001 C CNN
 F 3 "" H 4800 5475 50  0000 C CNN
 	1    4800 5475
@@
 F 0 "R17" V 4750 5375 50  0000 C CNN
 F 1 "1k" V 4750 5775 50  0000 C CNN
-F 2 "Resistors_THT:R_Axial_DIN0207_L6.3mm_D2.5mm_P10.16mm_Horizontal" V 4730 5575 50  0001 C CNN
+F 2 "Resistors_THT:R_Axial_DIN0411_L9.9mm_D3.6mm_P5.08mm_Vertical" V 4730 5575 50  0001 C CNN
 F 3 "" H 4800 5575 50  0000 C CNN
 	1    4800 5575
@@
 F 0 "R18" V 4750 5925 50  0000 C CNN
 F 1 "1k" V 4750 6325 50  0000 C CNN
-F 2 "Resistors_THT:R_Axial_DIN0207_L6.3mm_D2.5mm_P10.16mm_Horizontal" V 4730 6125 50  0001 C CNN
+F 2 "Resistors_THT:R_Axial_DIN0411_L9.9mm_D3.6mm_P5.08mm_Vertical" V 4730 6125 50  0001 C CNN
 F 3 "" H 4800 6125 50  0000 C CNN
 	1    4800 6125
@@
 P 2675 3450
 F 0 "D8" H 2800 3550 50  0000 C CNN
-F 1 "BY399" H 2450 3550 50  0000 C CNN
+F 1 "1N4001" H 2450 3550 50  0000 C CNN
 F 2 "Diodes_THT:D_A-405_P12.70mm_Horizontal" H 2675 3450 60  0001 C CNN
 F 3 "" H 2675 3450 60  0001 C CNN
@@
 P 2675 3250
 F 0 "D7" H 2800 3150 50  0000 C CNN
-F 1 "BY399" H 2450 3150 50  0000 C CNN
+F 1 "1N4001" H 2450 3150 50  0000 C CNN
 F 2 "Diodes_THT:D_A-405_P12.70mm_Horizontal" H 2675 3250 60  0001 C CNN
 F 3 "" H 2675 3250 60  0001 C CNN
@@
 F 0 "R3" V 5750 3150 50  0000 C CNN
 F 1 "40" V 5750 3300 50  0000 C CNN
-F 2 "Resistors_THT:R_Axial_DIN0414_L11.9mm_D4.5mm_P15.24mm_Horizontal" V 5780 3250 50  0001 C CNN
+F 2 "Resistors_THT:R_Axial_DIN0411_L9.9mm_D3.6mm_P12.70mm_Horizontal" V 5780 3250 50  0001 C CNN
 F 3 "" H 5850 3250 50  0000 C CNN
 	1    5850 3250
@@
 F 0 "R4" V 6350 3150 50  0000 C CNN
 F 1 "80" V 6350 3300 50  0000 C CNN
-F 2 "Resistors_THT:R_Axial_DIN0414_L11.9mm_D4.5mm_P15.24mm_Horizontal" V 6380 3250 50  0001 C CNN
+F 2 "Resistors_THT:R_Axial_DIN0411_L9.9mm_D3.6mm_P12.70mm_Horizontal" V 6380 3250 50  0001 C CNN
 F 3 "" H 6450 3250 50  0000 C CNN
 	1    6450 3250
@@
 F 0 "R7" V 8150 3150 50  0000 C CNN
 F 1 "640" V 8150 3300 50  0000 C CNN
-F 2 "Resistors_THT:R_Axial_DIN0414_L11.9mm_D4.5mm_P15.24mm_Horizontal" V 8180 3250 50  0001 C CNN
+F 2 "Resistors_THT:R_Axial_DIN0411_L9.9mm_D3.6mm_P12.70mm_Horizontal" V 8180 3250 50  0001 C CNN
 F 3 "" H 8250 3250 50  0000 C CNN
 	1    8250 3250
@@
 F 0 "R6" V 7550 3150 50  0000 C CNN
 F 1 "320" V 7550 3300 50  0000 C CNN
-F 2 "Resistors_THT:R_Axial_DIN0414_L11.9mm_D4.5mm_P15.24mm_Horizontal" V 7580 3250 50  0001 C CNN
+F 2 "Resistors_THT:R_Axial_DIN0411_L9.9mm_D3.6mm_P12.70mm_Horizontal" V 7580 3250 50  0001 C CNN
 F 3 "" H 7650 3250 50  0000 C CNN
 	1    7650 3250
@@
 F 0 "R5" V 6950 3150 50  0000 C CNN
 F 1 "160" V 6950 3300 50  0000 C CNN
-F 2 "Resistors_THT:R_Axial_DIN0414_L11.9mm_D4.5mm_P15.24mm_Horizontal" V 6980 3250 50  0001 C CNN
+F 2 "Resistors_THT:R_Axial_DIN0411_L9.9mm_D3.6mm_P12.70mm_Horizontal" V 6980 3250 50  0001 C CNN
 F 3 "" H 7050 3250 50  0000 C CNN
 	1    7050 3250
@@
 P 10200 4575
 F 0 "T9" H 10500 4575 50  0000 R CNN
-F 1 "BC109" H 10375 4200 50  0000 R CNN
+F 1 "BC109" H 10650 4450 50  0000 R CNN
 F 2 "TO_SOT_Packages_THT:TO-18-3" H 10200 4575 60  0001 C CNN
 F 3 "" H 10200 4575 60  0001 C CNN
@@
 Um3
 $Comp
-L GND-RESCUE-ctt #PWR02
+L GND-RESCUE-ctt #PWR03
 U 1 1 631FCAC7
 P 9950 2150
-F 0 "#PWR02" H 9950 2150 30  0001 C CNN
+F 0 "#PWR03" H 9950 2150 30  0001 C CNN
 F 1 "GND-RESCUE-ctt" H 9950 2080 30  0001 C CNN
 F 2 "" H 9950 2150 60  0001 C CNN
@@
 F 0 "R8" V 8750 3150 50  0000 C CNN
 F 1 "1280" V 8750 3350 50  0000 C CNN
-F 2 "Resistors_THT:R_Axial_DIN0414_L11.9mm_D4.5mm_P15.24mm_Horizontal" V 8780 3250 50  0001 C CNN
+F 2 "Resistors_THT:R_Axial_DIN0411_L9.9mm_D3.6mm_P12.70mm_Horizontal" V 8780 3250 50  0001 C CNN
 F 3 "" H 8850 3250 50  0000 C CNN
 	1    8850 3250
@@
 F 0 "R9" V 9350 3150 50  0000 C CNN
 F 1 "2560" V 9350 3350 50  0000 C CNN
-F 2 "Resistors_THT:R_Axial_DIN0414_L11.9mm_D4.5mm_P15.24mm_Horizontal" V 9380 3250 50  0001 C CNN
+F 2 "Resistors_THT:R_Axial_DIN0411_L9.9mm_D3.6mm_P12.70mm_Horizontal" V 9380 3250 50  0001 C CNN
 F 3 "" H 9450 3250 50  0000 C CNN
 	1    9450 3250
@@
 F 0 "D5" H 9275 2500 50  0000 C CNN
 F 1 "1N4001" H 9450 2650 50  0000 C CNN
-F 2 "Diodes_THT:D_A-405_P12.70mm_Horizontal" H 9450 2550 60  0001 C CNN
+F 2 "Diodes_THT:D_A-405_P10.16mm_Horizontal" H 9450 2550 60  0001 C CNN
 F 3 "" H 9450 2550 60  0001 C CNN
 	1    9450 2550
@@
 	10000 6125 10000 4575
 Wire Wire Line
-	10300 4875 10300 4775
+	10300 4775 10300 5225
 Wire Wire Line
 	5500 4875 10300 4875
@@
 Text Notes 10050 1900 0    60   ~ 0
 1
+$Comp
+L GND-RESCUE-ctt #PWR04
+U 1 1 6328D5D6
+P 10300 5225
+F 0 "#PWR04" H 10300 5225 30  0001 C CNN
+F 1 "GND-RESCUE-ctt" H 10300 5155 30  0001 C CNN
+F 2 "" H 10300 5225 60  0001 C CNN
+F 3 "" H 10300 5225 60  0001 C CNN
+	1    10300 5225
+	1    0    0    -1
+$EndComp
+Connection ~ 10300 4875
 $EndSCHEMATC

Commit message: 220920
Changed lines of the file:
@@
 EESchema Schematic File Version 2
-LIBS:ctt-rescue
 LIBS:power
 LIBS:device
+LIBS:transistors
 LIBS:conn
 LIBS:linear
@@
 LIBS:cypress
 LIBS:siliconi
+LIBS:opto
+LIBS:atmel
 LIBS:contrib
 LIBS:valves
 LIBS:ctt-cache
+LIBS:ctt-rescue
+LIBS:relay_leg-5
+LIBS:ctt_ps2-cache
 EELAYER 25 0
 EELAYER END
 $Descr A4 11693 8268
 encoding utf-8
-Sheet 4 11
+Sheet 1 1
 Title "CTT Transistor tester - CTT/PS2 power supply unit"
 Date "28 jan 2012"
@@
 $EndComp
 Text Notes 1650 4875 0    60   ~ 0
+2
+Text Notes 1650 4975 0    60   ~ 0
+4
+Text Notes 1650 5075 0    60   ~ 0
+6
+Text Notes 1650 5175 0    60   ~ 0
+8
+Text Notes 1650 5275 0    60   ~ 0
+7
+Text Notes 1650 5375 0    60   ~ 0
+5
+Text Notes 1650 5475 0    60   ~ 0
+3
+Text Notes 1650 5575 0    60   ~ 0
 1
-Text Notes 1650 4975 0    60   ~ 0
-2
-Text Notes 1650 5075 0    60   ~ 0
-3
-Text Notes 1650 5175 0    60   ~ 0
-4
-Text Notes 1650 5275 0    60   ~ 0
-5
-Text Notes 1650 5375 0    60   ~ 0
-6
-Text Notes 1650 5475 0    60   ~ 0
-7
-Text Notes 1650 5575 0    60   ~ 0
-8
 Text Notes 1650 1650 0    60   ~ 0
 1
