File: cad_files/ctt_ps3/ctt_ps3.kicad_pcb (KiCad board)
At the start: 2 copper layers, 141 x 73.7 mm, 0 parts

Commit message: 220920
Parts:
- added C1: 2200u, Capacitors_THT:CP_Radial_D14.0mm_P7.50mm, F.Cu at (97.8, 86.4)
- added C2: 10u, Capacitors_THT:CP_Radial_D5.0mm_P2.50mm, F.Cu at (114.3, 87.0)
- added C3: 10u, Capacitors_THT:CP_Radial_D5.0mm_P2.50mm, F.Cu at (114.3, 92.7)
- added C4: 470u, Capacitors_THT:CP_Radial_D10.0mm_P5.00mm, F.Cu at (104.1, 73.7)
- added C5: 100u, Capacitors_THT:CP_Radial_D10.0mm_P5.00mm, F.Cu at (116.2, 111.8)
- added C6: 100n, Capacitors_THT:C_Disc_D6.0mm_W2.5mm_P5.00mm, F.Cu at (109.2, 111.8)
- added CN1: Pin_Header_Straight_1x03, Pin_Headers:Pin_Header_Straight_1x03, F.Cu at (85.1, 66.0)
- added CN2: Pin_Header_Straight_1x02, Pin_Headers:Pin_Header_Straight_1x02, F.Cu at (118.1, 119.4)
- added CN3: Pin_Header_Straight_1x08, Pin_Headers:Pin_Header_Straight_1x08, F.Cu at (104.1, 96.5)
- added CN4: Pin_Header_Straight_1x01, Pin_Headers:Pin_Header_Straight_1x01, F.Cu at (81.3, 96.5)
- added CN5: Pin_Header_Straight_1x01, Pin_Headers:Pin_Header_Straight_1x01, F.Cu at (109.2, 96.5)
- added CN6: Pin_Header_Straight_1x01, Pin_Headers:Pin_Header_Straight_1x01, F.Cu at (118.1, 129.5)
- added D1: 1N4002, Diodes_THT:D_A-405_P12.70mm_Horizontal, F.Cu at (116.8, 69.8)
- added D10: 1N4001, Diodes_THT:D_A-405_P12.70mm_Horizontal, F.Cu at (171.4, 94.0)
- added D11: 1N4001, Diodes_THT:D_A-405_P12.70mm_Horizontal, F.Cu at (189.2, 94.0)
- added D12: 1N4001, Diodes_THT:D_A-405_P12.70mm_Horizontal, F.Cu at (207.0, 94.0)
- added D13: 1N4001, Diodes_THT:D_A-405_P12.70mm_Horizontal, F.Cu at (194.3, 99.1)
- added D14: 1N4001, Diodes_THT:D_A-405_P12.70mm_Horizontal, F.Cu at (176.5, 99.1)
- added D15: 1N4001, Diodes_THT:D_A-405_P12.70mm_Horizontal, F.Cu at (158.8, 99.1)
- added D16: 1N4001, Diodes_THT:D_A-405_P12.70mm_Horizontal, F.Cu at (141.0, 99.1)
- added D2: BY399, Diodes_THT:D_5W_P12.70mm_Horizontal, F.Cu at (83.8, 83.8)
- added D3: BY399, Diodes_THT:D_5W_P12.70mm_Horizontal, F.Cu at (88.9, 83.8)
- added D4: 1N4002, Diodes_THT:D_A-405_P12.70mm_Horizontal, F.Cu at (114.3, 69.8)
- added D5: 1N4001, Diodes_THT:D_A-405_P10.16mm_Horizontal, F.Cu at (111.8, 129.5)
- added D6: ZPD27, Diodes_THT:D_A-405_P12.70mm_Horizontal, F.Cu at (80.0, 88.9)
- added D7: 1N4001, Diodes_THT:D_A-405_P12.70mm_Horizontal, F.Cu at (80.0, 71.1)
- added D8: 1N4001, Diodes_THT:D_A-405_P12.70mm_Horizontal, F.Cu at (92.7, 71.1)
- added D9: 1N4001, Diodes_THT:D_A-405_P12.70mm_Horizontal, F.Cu at (153.7, 94.0)
- added IC1: LM317T, Power_Integrations:TO-220, F.Cu at (114.3, 66.0)
- added IC2: 74LS374, Housings_DIP:DIP-20_W7.62mm_LongPads, F.Cu at (104.1, 105.4)
- added K1: LMR2-5D, relay_lmr2:relay_lmr2, F.Cu at (94.0, 124.5)
- added K2: LEG-5, relay_leg:relay_leg, F.Cu at (147.3, 80.0)
- added K3: LEG-5, relay_leg:relay_leg, F.Cu at (165.1, 80.0)
- added K4: LEG-5, relay_leg:relay_leg, F.Cu at (182.9, 80.0)
- added K5: LEG-5, relay_leg:relay_leg, F.Cu at (200.7, 80.0)
- added K6: LEG-5, relay_leg:relay_leg, F.Cu at (200.7, 113.7)
- added K7: LEG-5, relay_leg:relay_leg, F.Cu at (182.9, 113.7)
- added K8: LEG-5, relay_leg:relay_leg, F.Cu at (165.1, 113.7)
- added K9: LEG-5, relay_leg:relay_leg, F.Cu at (147.3, 113.7)
- added P1: 390, Potentiometers:Potentiometer_WirePads_Small, F.Cu at (99.1, 66.0)
- added R1: 640, Resistors_THT:R_Axial_DIN0411_L9.9mm_D3.6mm_P12.70mm_Horizontal, F.Cu at (110.5, 82.5)
- added R10: 1k, Resistors_THT:R_Axial_DIN0411_L9.9mm_D3.6mm_P5.08mm_Vertical, F.Cu at (128.3, 88.9)
- added R11: 1k, Resistors_THT:R_Axial_DIN0411_L9.9mm_D3.6mm_P5.08mm_Vertical, F.Cu at (128.3, 81.3)
- added R12: 1k, Resistors_THT:R_Axial_DIN0411_L9.9mm_D3.6mm_P5.08mm_Vertical, F.Cu at (128.3, 73.7)
- added R13: 1k, Resistors_THT:R_Axial_DIN0411_L9.9mm_D3.6mm_P5.08mm_Vertical, F.Cu at (128.3, 66.0)
- added R14: 1k, Resistors_THT:R_Axial_DIN0411_L9.9mm_D3.6mm_P5.08mm_Vertical, F.Cu at (128.3, 119.4)
- added R15: 1k, Resistors_THT:R_Axial_DIN0411_L9.9mm_D3.6mm_P5.08mm_Vertical, F.Cu at (128.3, 111.8)
- added R16: 1k, Resistors_THT:R_Axial_DIN0411_L9.9mm_D3.6mm_P5.08mm_Vertical, F.Cu at (128.3, 104.1)
- added R17: 1k, Resistors_THT:R_Axial_DIN0411_L9.9mm_D3.6mm_P5.08mm_Vertical, F.Cu at (128.3, 96.5)
- added R18: 1k, Resistors_THT:R_Axial_DIN0411_L9.9mm_D3.6mm_P5.08mm_Vertical, F.Cu at (128.3, 127.0)
- added R2: 2, Resistors_THT:R_Axial_DIN0411_L9.9mm_D3.6mm_P12.70mm_Horizontal, F.Cu at (153.7, 66.0)
- added R3: 4, Resistors_THT:R_Axial_DIN0411_L9.9mm_D3.6mm_P12.70mm_Horizontal, F.Cu at (171.4, 66.0)
- added R4: 8, Resistors_THT:R_Axial_DIN0411_L9.9mm_D3.6mm_P12.70mm_Horizontal, F.Cu at (189.2, 66.0)
- added R5: 16, Resistors_THT:R_Axial_DIN0411_L9.9mm_D3.6mm_P12.70mm_Horizontal, F.Cu at (207.0, 66.0)
- added R6: 32, Resistors_THT:R_Axial_DIN0411_L9.9mm_D3.6mm_P12.70mm_Horizontal, F.Cu at (194.3, 128.3)
- added R7: 64, Resistors_THT:R_Axial_DIN0411_L9.9mm_D3.6mm_P12.70mm_Horizontal, F.Cu at (176.5, 128.3)
- added R8: 128, Resistors_THT:R_Axial_DIN0411_L9.9mm_D3.6mm_P12.70mm_Horizontal, F.Cu at (158.8, 128.3)
- added R9: 256, Resistors_THT:R_Axial_DIN0411_L9.9mm_D3.6mm_P12.70mm_Horizontal, F.Cu at (141.0, 128.3)
- added T1: BC109, TO_SOT_Packages_THT:TO-18-3, F.Cu at (134.6, 90.2)
- added T2: BC109, TO_SOT_Packages_THT:TO-18-3, F.Cu at (134.6, 82.5)
- added T3: BC109, TO_SOT_Packages_THT:TO-18-3, F.Cu at (134.6, 74.9)
- added T4: BC109, TO_SOT_Packages_THT:TO-18-3, F.Cu at (134.6, 67.3)
- added T5: BC109, TO_SOT_Packages_THT:TO-18-3, F.Cu at (134.6, 120.7)
- added T6: BC109, TO_SOT_Packages_THT:TO-18-3, F.Cu at (134.6, 113.0)
- added T7: BC109, TO_SOT_Packages_THT:TO-18-3, F.Cu at (134.6, 105.4)
- added T8: BC109, TO_SOT_Packages_THT:TO-18-3, F.Cu at (134.6, 97.8)
- added T9: BC109, TO_SOT_Packages_THT:TO-18-3, F.Cu at (134.6, 128.3)
Routing:
- net GND: track 0.00 -> 196.0 mm
- net Net-(C3-Pad1): track 0.00 -> 133.2 mm, vias 0 -> 1
- net Net-(C2-Pad1): track 0.00 -> 118.5 mm
- net VCC: track 0.00 -> 116.7 mm
- net /5V 100mA AC COM: track 0.00 -> 115.5 mm
- net Net-(D12-Pad2): track 0.00 -> 108.0 mm
- net Net-(D9-Pad2): track 0.00 -> 107.8 mm
- net Net-(K5-Pad3): track 0.00 -> 96.6 mm
- net Net-(D11-Pad2): track 0.00 -> 83.4 mm
- net Net-(IC2-Pad9): track 0.00 -> 73.5 mm, vias 0 -> 1
- net Net-(D13-Pad2): track 0.00 -> 69.5 mm
- net Net-(IC2-Pad6): track 0.00 -> 59.0 mm, vias 0 -> 1
- net Net-(D6-Pad2): track 0.00 -> 57.2 mm
- net Net-(D10-Pad2): track 0.00 -> 56.9 mm
- net Net-(D14-Pad2): track 0.00 -> 54.8 mm
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Other:
- board text added: "CTT/PS2-3"
- board text added: "DN: CTT/25-27"
- board text added: "http://www.pozsarzs.hu"
