File: cad_files/ctt_ps3/ctt_ps3.kicad_pcb (KiCad board)
At the start: 2 copper layers, 141 x 73.7 mm, 67 parts, among them CN1 Pin_Header_Straight_1x03, CN2 Pin_Header_Straight_1x02, CN3 Pin_Header_Straight_1x08, CN4 Pin_Header_Straight_1x01, CN5 Pin_Header_Straight_1x01, CN6 Pin_Header_Straight_1x01, IC1 LM317T, IC2 74LS374, K1 LMR2-5D, K2 LEG-5, K3 LEG-5, K4 LEG-5, K5 LEG-5, K6 LEG-5, K7 LEG-5, K8 LEG-5, K9 LEG-5, P1 390, T1 BC109, T2 BC109, T3 BC109, T4 BC109, T5 BC109, T6 BC109, T7 BC109, T8 BC109, T9 BC109

Commit message: 220928
Parts:
- IC1: value LM317T -> LM317L
Changed lines of the file:
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@@
       (effects (font (size 1 1) (thickness 0.15)))
     )
-    (fp_text value LM317T (at 0 -4.318) (layer F.Fab)
+    (fp_text value LM317L (at 0 -4.318) (layer F.Fab)
       (effects (font (size 1 1) (thickness 0.15)))
     )
