File: cad_files/ctt_ps3/ctt_ps3.sch (KiCad schematic (older format))
At the start: 61 parts, among them IC1 LM317L, IC2 74LS374, K1 LMR2-5D, K2 LEG-5, K3 LEG-5, K4 LEG-5, K5 LEG-5, K6 LEG-5, K7 LEG-5, K8 LEG-5, K9 LEG-5, P1 390, T1 BC109, T2 BC109, T3 BC109, T4 BC109, T5 BC109, T6 BC109, T7 BC109, T8 BC109, T9 BC109

Commit message: 220915
Other:
- note added: "1"
- note added: "2"
- note added: "3"
- note added: "4"
- note added: "5"
- note added: "6"
- note added: "7"
- note added: "8"
Changed lines of the file:
@@
 $EndComp
 Connection ~ 3600 3750
+Text Notes 10050 1900 0    60   ~ 0
+1
+Text Notes 1650 1650 0    60   ~ 0
+1
+Text Notes 1650 2550 0    60   ~ 0
+3
+Text Notes 1650 3450 0    60   ~ 0
+2
+Text Notes 1650 3750 0    60   ~ 0
+1
+Text Notes 1650 4350 0    60   ~ 0
+2
+Text Notes 1650 4875 0    60   ~ 0
+1
+Text Notes 1650 4975 0    60   ~ 0
+2
+Text Notes 1650 5075 0    60   ~ 0
+3
+Text Notes 1650 5175 0    60   ~ 0
+4
+Text Notes 1650 5275 0    60   ~ 0
+5
+Text Notes 1650 5375 0    60   ~ 0
+6
+Text Notes 1650 5475 0    60   ~ 0
+7
+Text Notes 1650 5575 0    60   ~ 0
+8
+Text Notes 1650 5775 0    60   ~ 0
+1
+Text Notes 1650 6125 0    60   ~ 0
+1
 $EndSCHEMATC

Commit message: 220919
Connections:
- net GND: now also T1.1 (E), T2.1 (E), T3.1 (E), T4.1 (E), T5.1 (E), T6.1 (E), T7.1 (E), T8.1 (E), T9.1 (E)
Changed lines of the file:
@@
 Rev "1.0"
 Comp "Pozsar Zsolt"
-Comment1 "Draw number: CTT/37"
+Comment1 "Draw number: CTT/28"
 Comment2 ""
 Comment3 ""
@@
 P 10200 4575
 F 0 "T9" H 10500 4575 50  0000 R CNN
-F 1 "BC109" H 10375 4200 50  0000 R CNN
+F 1 "BC109" H 10650 4475 50  0000 R CNN
 F 2 "" H 10200 4575 60  0001 C CNN
 F 3 "" H 10200 4575 60  0001 C CNN
@@
 Text Notes 1650 6125 0    60   ~ 0
 1
+$Comp
+L GND-RESCUE-ctt #PWR?
+U 1 1 6328FABE
+P 10300 5225
+F 0 "#PWR?" H 10300 5225 30  0001 C CNN
+F 1 "GND-RESCUE-ctt" H 10300 5155 30  0001 C CNN
+F 2 "" H 10300 5225 60  0001 C CNN
+F 3 "" H 10300 5225 60  0001 C CNN
+	1    10300 5225
+	1    0    0    -1
+$EndComp
+Wire Wire Line
+	10300 4875 10300 5225
+Connection ~ 10300 4875
 $EndSCHEMATC

Commit message: 220920
Parts:
- C1: value 470u -> 2200u; footprint (none) -> Capacitors_THT:CP_Radial_D14.0mm_P7.50mm
- C2, C3: footprint (none) -> Capacitors_THT:CP_Radial_D5.0mm_P2.50mm
- C4, C5: footprint (none) -> Capacitors_THT:CP_Radial_D10.0mm_P5.00mm
- C6: footprint (none) -> Capacitors_THT:C_Disc_D6.0mm_W2.5mm_P5.00mm
- D1, D10, D11, D12, D13, D14, D15, D16, D4, D7, D8, D9: footprint (none) -> Diodes_THT:D_A-405_P12.70mm_Horizontal
- D2, D3: value 1N4001 -> BY399; footprint (none) -> Diodes_THT:D_5W_P12.70mm_Horizontal
- D5: footprint (none) -> Diodes_THT:D_A-405_P10.16mm_Horizontal
- D6: value ZPD3,3 -> ZPD27; footprint (none) -> Diodes_THT:D_A-405_P12.70mm_Horizontal
- IC1: value LM317L -> LM317T; footprint TO-92 -> Power_Integrations:TO-220
- IC2: footprint (none) -> Housings_DIP:DIP-20_W7.62mm_LongPads
- K1: footprint (none) -> relay_lmr2:relay_lmr2
- K2, K3, K4, K5, K6, K7, K8, K9: footprint (none) -> relay_leg:relay_leg
- P1: footprint (none) -> Potentiometers:Potentiometer_WirePads_Small
- R1, R2, R3, R4, R5, R6, R7, R8, R9: footprint (none) -> Resistors_THT:R_Axial_DIN0411_L9.9mm_D3.6mm_P12.70mm_Horizontal
- R10, R11, R12, R13, R14, R15, R16, R17, R18: footprint (none) -> Resistors_THT:R_Axial_DIN0411_L9.9mm_D3.6mm_P5.08mm_Vertical
- T1, T2, T3, T4, T5, T6, T7, T8, T9: footprint (none) -> TO_SOT_Packages_THT:TO-18-3
Connections:
- net Um1 renamed Um3

Commit message: 220928
Parts:
- IC1: value LM317T -> LM317L
Changed lines of the file:
@@
 EESchema Schematic File Version 2
+LIBS:ctt-rescue
 LIBS:power
 LIBS:device
-LIBS:transistors
 LIBS:conn
 LIBS:linear
@@
 LIBS:cypress
 LIBS:siliconi
-LIBS:opto
-LIBS:atmel
 LIBS:contrib
 LIBS:valves
 LIBS:ctt-cache
-LIBS:ctt-rescue
-LIBS:relay_leg-5
-LIBS:ctt_ps3-cache
 EELAYER 25 0
 EELAYER END
 $Descr A4 11693 8268
 encoding utf-8
-Sheet 1 1
+Sheet 2 11
 Title "CTT Transistor tester - CTT/PS3 power supply unit"
 Date "28 jan 2012"
@@
 P 3700 1700
 F 0 "IC1" H 3500 1900 50  0000 C CNN
-F 1 "LM317T" H 3700 1900 50  0000 L CNN
+F 1 "LM317L" H 3700 1900 50  0000 L CNN
 F 2 "Power_Integrations:TO-220" H 3700 1800 50  0001 C CIN
 F 3 "" H 3700 1700 50  0000 C CNN
@@
 Connection ~ 9800 3500
 Wire Wire Line
-	9800 4300 3700 4300
+	3700 4300 9800 4300
 Wire Wire Line
 	9700 2850 10300 2850
@@
 	9200 3000 9900 3000
 Wire Wire Line
-	9900 4150 9900 3000
+	9900 3000 9900 4150
 Wire Wire Line
 	10300 2850 10300 4375
@@
 Connection ~ 9200 4000
 Wire Wire Line
-	5000 4150 9900 4150
-Wire Wire Line
-	9800 3250 9800 4300
+	9900 4150 5000 4150
+Wire Wire Line
+	9800 4300 9800 3250
 Wire Wire Line
 	9700 4000 9650 4000

Commit message: 220928
Parts:
- D1, D4: value 1N4002 -> 1N4001
- D2, D3: value BY399 -> 1N4001
- D6: value ZPD27 -> ZPD3
Changed lines of the file:
@@
 $Comp
 L 74LS374 IC2
-U 1 1 631D5E1D
+U 1 1 63341076
 P 3850 5375
 F 0 "IC2" H 3850 5375 60  0000 C CNN
@@
 $Comp
 L CP-RESCUE-ctt C1
-U 1 1 4DE6513B
+U 1 1 63341074
 P 3200 2050
 F 0 "C1" H 3250 2200 50  0000 L CNN
@@
 $Comp
 L CP-RESCUE-ctt C2
-U 1 1 4DE65139
+U 1 1 63341073
 P 4600 2050
 F 0 "C2" H 4700 2200 50  0000 L CNN
@@
 $Comp
 L DIODE D3
-U 1 1 4DE65132
+U 1 1 63341072
 P 2675 1850
 F 0 "D3" H 2550 1950 50  0000 C CNN
-F 1 "BY399" H 2850 1950 50  0000 C CNN
+F 1 "1N4001" H 2850 1950 50  0000 C CNN
 F 2 "Diodes_THT:D_5W_P12.70mm_Horizontal" H 2675 1850 60  0001 C CNN
 F 3 "" H 2675 1850 60  0001 C CNN
@@
 P 2675 1650
 F 0 "D2" H 2550 1550 50  0000 C CNN
-F 1 "BY399" H 2850 1550 50  0000 C CNN
+F 1 "1N4001" H 2850 1550 50  0000 C CNN
 F 2 "Diodes_THT:D_5W_P12.70mm_Horizontal" H 2675 1650 60  0001 C CNN
 F 3 "" H 2675 1650 60  0001 C CNN
@@
 $Comp
 L LM317T IC1
-U 1 1 631FCAA5
+U 1 1 63341088
 P 3700 1700
 F 0 "IC1" H 3500 1900 50  0000 C CNN
@@
 $Comp
 L DIODE D4
-U 1 1 631D5DA0
+U 1 1 63341075
 P 4000 2250
 F 0 "D4" H 3850 2350 50  0000 C CNN
-F 1 "1N4002" H 4000 2100 50  0000 C CNN
+F 1 "1N4001" H 4000 2100 50  0000 C CNN
 F 2 "Diodes_THT:D_A-405_P12.70mm_Horizontal" H 4000 2250 60  0001 C CNN
 F 3 "" H 4000 2250 60  0001 C CNN
@@
 $Comp
 L DIODE D1
-U 1 1 631FCAA9
+U 1 1 6334108A
 P 3700 1300
 F 0 "D1" H 3850 1250 50  0000 C CNN
-F 1 "1N4002" H 3700 1450 50  0000 C CNN
+F 1 "1N4001" H 3700 1450 50  0000 C CNN
 F 2 "Diodes_THT:D_A-405_P12.70mm_Horizontal" H 3700 1300 60  0001 C CNN
 F 3 "" H 3700 1300 60  0001 C CNN
@@
 $Comp
 L NPN T2
-U 1 1 631FCABA
+U 1 1 63341095
 P 6000 4575
 F 0 "T2" H 6300 4575 50  0000 R CNN
@@
 $Comp
 L NPN T3
-U 1 1 631DE0CA
+U 1 1 6334107D
 P 6600 4575
 F 0 "T3" H 6900 4575 50  0000 R CNN
@@
 $Comp
 L R R1
-U 1 1 631FCACC
+U 1 1 6334109D
 P 4000 2050
 F 0 "R1" V 3900 1950 50  0000 C CNN
@@
 $Comp
 L R R11
-U 1 1 631FCAD6
+U 1 1 633410A0
 P 4800 4975
 F 0 "R11" V 4750 4775 50  0000 C CNN
@@
 $Comp
 L R R12
-U 1 1 631FCAD7
+U 1 1 633410A1
 P 4800 5075
 F 0 "R12" V 4750 4875 50  0000 C CNN
@@
 $Comp
 L R R17
-U 1 1 631FCADC
+U 1 1 633410A5
 P 4800 5575
 F 0 "R17" V 4750 5375 50  0000 C CNN
@@
 $Comp
 L ZENER D6
-U 1 1 6321501A
+U 1 1 633410AF
 P 4250 3200
 F 0 "D6" H 4400 3100 50  0000 C CNN
-F 1 "ZPD27" H 4250 3350 50  0000 C CNN
+F 1 "ZPD3" H 4250 3350 50  0000 C CNN
 F 2 "Diodes_THT:D_A-405_P12.70mm_Horizontal" H 4250 3200 60  0001 C CNN
 F 3 "" H 4250 3200 60  0001 C CNN
@@
 +5V
 $Comp
-L GND-RESCUE-ctt #PWR01
+L GND-RESCUE-ctt #PWR09
 U 1 1 631FCAC6
 P 2150 4475
-F 0 "#PWR01" H 2150 4475 30  0001 C CNN
+F 0 "#PWR09" H 2150 4475 30  0001 C CNN
 F 1 "GND-RESCUE-ctt" H 2150 4405 30  0001 C CNN
 F 2 "" H 2150 4475 60  0001 C CNN
@@
 $EndComp
 $Comp
-L GND-RESCUE-ctt #PWR02
+L GND-RESCUE-ctt #PWR010
 U 1 1 631FCAC8
 P 3550 6275
-F 0 "#PWR02" H 3550 6275 30  0001 C CNN
+F 0 "#PWR010" H 3550 6275 30  0001 C CNN
 F 1 "GND-RESCUE-ctt" H 3550 6205 30  0001 C CNN
 F 2 "" H 3550 6275 60  0001 C CNN
@@
 $Comp
 L R R3
-U 1 1 632040F5
+U 1 1 633410A6
 P 5850 3250
 F 0 "R3" V 5750 3150 50  0000 C CNN
@@
 $Comp
 L Relay_LEG-5 K4
-U 1 1 631FCAAD
+U 1 1 6334108E
 P 6450 3650
 F 0 "K4" V 6450 3450 50  0000 L CNN
@@
 $Comp
 L CP-RESCUE-ctt C3
-U 1 1 631FC190
+U 1 1 63341085
 P 3450 2300
 F 0 "C3" H 3300 2450 50  0000 L CNN
@@
 $Comp
 L DIODE D14
-U 1 1 631FCAB7
+U 1 1 63341093
 P 8250 4000
 F 0 "D14" H 8100 3950 50  0000 C CNN
@@
 $Comp
 L DIODE D12
-U 1 1 631DAAD0
+U 1 1 6334107A
 P 7050 4000
 F 0 "D12" H 6900 3950 50  0000 C CNN
@@
 $Comp
 L Relay_LEG-5 K7
-U 1 1 631FCAB0
+U 1 1 63341091
 P 8250 3650
 F 0 "K7" V 8250 3450 50  0000 L CNN
@@
 $Comp
 L Relay_LEG-5 K6
-U 1 1 631FCAAF
+U 1 1 63341090
 P 7650 3650
 F 0 "K6" V 7650 3450 50  0000 L CNN
@@
 $Comp
 L R R7
-U 1 1 63204644
+U 1 1 633410A9
 P 8250 3250
 F 0 "R7" V 8150 3150 50  0000 C CNN
@@
 $Comp
 L R R6
-U 1 1 631FCAD0
+U 1 1 6334109E
 P 7650 3250
 F 0 "R6" V 7550 3150 50  0000 C CNN
@@
 $Comp
 L R R5
-U 1 1 6320433F
+U 1 1 633410A8
 P 7050 3250
 F 0 "R5" V 6950 3150 50  0000 C CNN
@@
 $Comp
 L NPN T6
-U 1 1 631FCABE
+U 1 1 63341096
 P 8400 4575
 F 0 "T6" H 8700 4575 50  0000 R CNN
@@
 Um3
 $Comp
-L GND-RESCUE-ctt #PWR03
-U 1 1 631FCAC7
+L GND-RESCUE-ctt #PWR011
+U 1 1 6334109B
 P 9950 2150
-F 0 "#PWR03" H 9950 2150 30  0001 C CNN
+F 0 "#PWR011" H 9950 2150 30  0001 C CNN
 F 1 "GND-RESCUE-ctt" H 9950 2080 30  0001 C CNN
 F 2 "" H 9950 2150 60  0001 C CNN
@@
 $Comp
 L R R8
-U 1 1 63204751
+U 1 1 633410AA
 P 8850 3250
 F 0 "R8" V 8750 3150 50  0000 C CNN
@@
 $Comp
 L Relay_LEG-5 K9
-U 1 1 631D9D74
+U 1 1 63341077
 P 9450 3650
 F 0 "K9" V 9450 3450 50  0000 L CNN
@@
 $Comp
 L DIODE D15
-U 1 1 631FCAB8
+U 1 1 63341094
 P 8850 4000
 F 0 "D15" H 8700 3950 50  0000 C CNN
@@
 $Comp
 L DIODE D5
-U 1 1 631FCAC5
+U 1 1 63341099
 P 9450 2550
 F 0 "D5" H 9275 2500 50  0000 C CNN
@@
 1
 $Comp
-L GND-RESCUE-ctt #PWR04
-U 1 1 6328D5D6
+L GND-RESCUE-ctt #PWR012
+U 1 1 633410B2
 P 10300 5225
-F 0 "#PWR04" H 10300 5225 30  0001 C CNN
+F 0 "#PWR012" H 10300 5225 30  0001 C CNN
 F 1 "GND-RESCUE-ctt" H 10300 5155 30  0001 C CNN
 F 2 "" H 10300 5225 60  0001 C CNN
